Commit message: FIXED FIXED FIXED

File: src/sec_bot/description/ros2_control.xacro (robot description, xacro)
@@ -13,5 +13,6 @@
                 <param name="enc_counts_per_rev">3436</param>
             </hardware>
-            <joint name="left_wheel_joint">
+            <!-- Front Left Wheel -->
+            <joint name="left_front_wheel_joint">
                 <command_interface name="velocity">
                     <param name="min">-10</param>
@@ -21,5 +22,24 @@
                 <state_interface name="position"/>
             </joint>
-            <joint name="right_wheel_joint">
+            <!-- Back Left Wheel -->
+            <joint name="left_back_wheel_joint">
+                <command_interface name="velocity">
+                    <param name="min">-10</param>
+                    <param name="max">10</param>
+                </command_interface>
+                <state_interface name="velocity"/>
+                <state_interface name="position"/>
+            </joint>
+            <!-- Front Right Wheel -->
+            <joint name="right_front_wheel_joint">
+                <command_interface name="velocity">
+                    <param name="min">-10</param>
+                    <param name="max">10</param>
+                </command_interface>
+                <state_interface name="velocity"/>
+                <state_interface name="position"/>
+            </joint>
+            <!-- Back Right Wheel -->
+            <joint name="right_back_wheel_joint">
                 <command_interface name="velocity">
                     <param name="min">-10</param>
@@ -36,17 +56,22 @@
                 <plugin>gazebo_ros2_control/GazeboSystem</plugin>
             </hardware>
-            <joint name="left_wheel_joint">
-                <command_interface name="velocity">
-                    <param name="min">-10</param>
-                    <param name="max">10</param>
-                </command_interface>
+            <!-- Identical joint declarations for simulation -->
+            <joint name="left_front_wheel_joint">
+                <command_interface name="velocity"/>
                 <state_interface name="velocity"/>
                 <state_interface name="position"/>
             </joint>
-            <joint name="right_wheel_joint">
-                <command_interface name="velocity">
-                    <param name="min">-10</param>
-                    <param name="max">10</param>
-                </command_interface>
+            <joint name="left_back_wheel_joint">
+                <command_interface name="velocity"/>
+                <state_interface name="velocity"/>
+                <state_interface name="position"/>
+            </joint>
+            <joint name="right_front_wheel_joint">
+                <command_interface name="velocity"/>
+                <state_interface name="velocity"/>
+                <state_interface name="position"/>
+            </joint>
+            <joint name="right_back_wheel_joint">
+                <command_interface name="velocity"/>
                 <state_interface name="velocity"/>
                 <state_interface name="position"/>
