Commit message: revert inertial_macros.xacro to working form

File: src/sec_bot/description/inertial_macros.xacro (robot description, xacro)
@@ -1,33 +1,32 @@
 <?xml version="1.0"?>
-<robot xmlns:xacro="http://www.ros.org/wiki/xacro">
-  <!-- box inertial macro with explicit origin parameters -->
-  <xacro:macro name="inertial_box"
-               params="mass:=1.0 x:=0.1 y:=0.1 z:=0.1
-                       origin_xyz:=0 0 0 origin_rpy:=0 0 0">
-    <inertial>
-      <origin xyz="${origin_xyz}" rpy="${origin_rpy}"/>
-      <mass value="${mass}"/>
-      <inertia
-        ixx="${mass*(y*y + z*z)/12}" ixy="0" ixz="0"
-        iyy="${mass*(x*x + z*z)/12}" iyz="0"
-        izz="${mass*(x*x + y*y)/12}"
-      />
-    </inertial>
-  </xacro:macro>
-  <!-- cylinder inertial macro with explicit origin parameters -->
-  <xacro:macro name="inertial_cylinder"
-               params="mass:=1.0 radius:=0.1 length:=0.1
-                       origin_xyz:=0 0 0 origin_rpy:=0 0 0">
-    <inertial>
-      <origin xyz="${origin_xyz}" rpy="${origin_rpy}"/>
-      <mass value="${mass}"/>
-      <inertia
-        ixx="${mass*(3*radius*radius + length*length)/12}"
-        ixy="0" ixz="0"
-        iyy="${mass*(3*radius*radius + length*length)/12}"
-        iyz="0"
-        izz="${mass*radius*radius/2}"
-      />
-    </inertial>
-  </xacro:macro>
-</robot>
+ <robot xmlns:xacro="http://www.ros.org/wiki/xacro" >
+     <!-- Specify some standard inertial calculations https://en.wikipedia.org/wiki/List_of_moments_of_inertia -->
+     <!-- These make use of xacro's mathematical functionality -->
+     <xacro:macro name="inertial_sphere" params="mass radius *origin">
+         <inertial>
+             <xacro:insert_block name="origin"/>
+             <mass value="${mass}" />
+             <inertia ixx="${(2/5) * mass * (radius*radius)}" ixy="0.0" ixz="0.0"
+                     iyy="${(2/5) * mass * (radius*radius)}" iyz="0.0"
+                     izz="${(2/5) * mass * (radius*radius)}" />
+         </inertial>
+     </xacro:macro>
+     <xacro:macro name="inertial_box" params="mass x y z *origin">
+         <inertial>
+             <xacro:insert_block name="origin"/>
+             <mass value="${mass}" />
+             <inertia ixx="${(1/12) * mass * (y*y+z*z)}" ixy="0.0" ixz="0.0"
+                     iyy="${(1/12) * mass * (x*x+z*z)}" iyz="0.0"
+                     izz="${(1/12) * mass * (x*x+y*y)}" />
+         </inertial>
+     </xacro:macro>
+     <xacro:macro name="inertial_cylinder" params="mass length radius *origin">
+         <inertial>
+             <xacro:insert_block name="origin"/>
+             <mass value="${mass}" />
+             <inertia ixx="${(1/12) * mass * (3*radius*radius + length*length)}" ixy="0.0" ixz="0.0"
+                     iyy="${(1/12) * mass * (3*radius*radius + length*length)}" iyz="0.0"
+                     izz="${(1/2) * mass * (radius*radius)}" />
+         </inertial>
+     </xacro:macro>
+ </robot>

Commit message: yeah enclosded shii and added red

File: src/sec_bot/description/inertial_macros.xacro (robot description, xacro)
@@ -1,4 +1,8 @@
 <?xml version="1.0"?>
 <robot xmlns:xacro="http://www.ros.org/wiki/xacro">
+  <!-- missing red material lol -->
+  <material name="red">
+    <color rgba="1 0 0 1"/>  <!-- Red color (R=1, G=0, B=0, Alpha=1) -->
+  </material>
   <!-- box inertial macro with explicit origin parameters -->
   <xacro:macro name="inertial_box"
@@ -18,5 +22,5 @@
   <xacro:macro name="inertial_cylinder"
                params="mass:=1.0 radius:=0.1 length:=0.1
-                       origin_xyz:=0 0 0 origin_rpy:=0 0 0">
+                       origin_xyz:='0 0 0 origin_rpy:=0 0 0'">
     <inertial>
       <origin xyz="${origin_xyz}" rpy="${origin_rpy}"/>

Commit message: updated inertial with peytons

File: src/sec_bot/description/inertial_macros.xacro (robot description, xacro)
@@ -31,3 +31,13 @@
     </inertial>
   </xacro:macro>
+  <!-- sphere inertial macro with explicit origin parameters -->
+  <xacro:macro name="inertial_sphere" params="mass radius *origin">
+      <inertial>
+          <xacro:insert_block name="origin"/>
+          <mass value="${mass}" />
+          <inertia ixx="${(2/5) * mass * (radius*radius)}" ixy="0.0" ixz="0.0"
+                  iyy="${(2/5) * mass * (radius*radius)}" iyz="0.0"
+                  izz="${(2/5) * mass * (radius*radius)}" />
+      </inertial>
+    </xacro:macro>
 </robot>

Commit message: testing something

File: src/sec_bot/description/inertial_macros.xacro (robot description, xacro)
@@ -40,4 +40,4 @@
                   izz="${(2/5) * mass * (radius*radius)}" />
       </inertial>
-    </xacro:macro>
+  </xacro:macro>
 </robot>

File: src/sec_bot/description/robot_core.xacro (robot description, xacro)
@@ -25,5 +25,5 @@
     <parent link="base_link"/>
     <child link="chassis"/>
-    <origin xyz="-0.1 0 0"/>
+    <origin xyz="5 0 0"/>
   </joint>
 <link name="chassis">
