Commit message: updated camera.xacro with peytons

File: src/sec_bot/description/camera.xacro (robot description, xacro)
@@ -14,2 +14,74 @@
         </visual>
     </link>
+    <joint name="camera_optical_joint" type="fixed">
+        <parent link="camera_link"/>
+        <child link="camera_link_optical"/>
+        <origin xyz="0 0 0" rpy="${-pi/2} 0 ${-pi/2}"/>
+    </joint>
+    <link name="camera_link_optical"></link>
+    <gazebo reference="camera_link">
+        <material>Gazebo/Red</material>
+        <sensor name="camera" type="camera">
+            <pose> 0 0 0 0 0 0 </pose>
+            <visualize>true</visualize>
+            <update_rate>10</update_rate>
+            <camera>
+                <horizontal_fov>1.089</horizontal_fov>
+                <image>
+                    <format>R8G8B8</format>
+                    <width>640</width>
+                    <height>480</height>
+                </image>
+                <clip>
+                    <near>0.05</near>
+                    <far>8.0</far>
+                </clip>
+            </camera>
+            <plugin name="camera_controller" filename="libgazebo_ros_camera.so">
+                <frame_name>camera_link_optical</frame_name>
+            </plugin>
+        </sensor>
+    </gazebo>
+    <joint name="camera2_joint" type="fixed">
+        <parent link="chassis"/>
+        <child link="camera2_link"/>
+        <origin xyz="0.32 -0.1400242 0.25" rpy="0 0 0"/>
+    </joint>
+    <link name="camera2_link">
+        <visual>
+            <geometry>
+                <box size="0.010 0.03 0.03"/>
+            </geometry>
+            <material name="red"/>
+        </visual>
+    </link>
+    <joint name="camera2_optical_joint" type="fixed">
+        <parent link="camera2_link"/>
+        <child link="camera2_link_optical"/>
+        <origin xyz="0 0 0" rpy="${-pi/2} 0 ${-pi/2}"/>
+    </joint>
+    <link name="camera2_link_optical"></link>
+    <gazebo reference="camera2_link">
+        <material>Gazebo/Red</material>
+        <sensor name="camera2" type="camera">
+            <pose> 0 0 0 0 0 0 </pose>
+            <visualize>true</visualize>
+            <update_rate>10</update_rate>
+            <camera>
+                <horizontal_fov>1.089</horizontal_fov>
+                <image>
+                    <format>R8G8B8</format>
+                    <width>640</width>
+                    <height>480</height>
+                </image>
+                <clip>
+                    <near>0.05</near>
+                    <far>8.0</far>
+                </clip>
+            </camera>
+            <plugin name="camera2_controller" filename="libgazebo_ros_camera.so">
+                <frame_name>camera2_link_optical</frame_name>
+            </plugin>
+        </sensor>
+    </gazebo>
+</robot>

Commit message: added inertial for camera link

File: src/sec_bot/description/camera.xacro (robot description, xacro)
@@ -12,5 +12,9 @@
             </geometry>
             <material name="red"/>
-        </visual>
+          </visual>
+          <inertial>
+              <mass value="0.001"/>
+              <inertia ixx="1e-6" ixy="0" ixz="0" iyy="1e-6" iyz="0" izz="1e-6"/>
+          </inertial>
     </link>
     <joint name="camera_optical_joint" type="fixed">

Commit message: added the same for camera2_LINK

File: src/sec_bot/description/camera.xacro (robot description, xacro)
@@ -59,4 +59,8 @@
             <material name="red"/>
         </visual>
+        <inertial>
+            <mass value="0.001"/>
+            <inertia ixx="1e-6" ixy="0" ixz="0" iyy="1e-6" iyz="0" izz="1e-6"/>
+        </inertial>
     </link>
     <joint name="camera2_optical_joint" type="fixed">

Commit message: yeah ahahahaha

File: src/sec_bot/description/camera.xacro (robot description, xacro)
@@ -1,87 +1,70 @@
 <?xml version="1.0"?>
-<robot xmlns:xacro="http://www.ros.org/wiki/xacro" >
-    <joint name="camera_joint" type="fixed">
-        <parent link="chassis"/>
-        <child link="camera_link"/>
-        <origin xyz="0.32 0.1400242 0.25" rpy="0 0 0"/>
-    </joint>
-    <link name="camera_link">
-        <visual>
-            <geometry>
-                <box size="0.010 0.03 0.03"/>
-            </geometry>
-            <material name="red"/>
-        </visual>
-    </link>
-    <joint name="camera_optical_joint" type="fixed">
-        <parent link="camera_link"/>
-        <child link="camera_link_optical"/>
-        <origin xyz="0 0 0" rpy="${-pi/2} 0 ${-pi/2}"/>
-    </joint>
-    <link name="camera_link_optical"></link>
-    <gazebo reference="camera_link">
-        <material>Gazebo/Red</material>
-        <sensor name="camera" type="camera">
-            <pose> 0 0 0 0 0 0 </pose>
-            <visualize>true</visualize>
-            <update_rate>10</update_rate>
-            <camera>
-                <horizontal_fov>1.089</horizontal_fov>
-                <image>
-                    <format>R8G8B8</format>
-                    <width>640</width>
-                    <height>480</height>
-                </image>
-                <clip>
-                    <near>0.05</near>
-                    <far>8.0</far>
-                </clip>
-            </camera>
-            <plugin name="camera_controller" filename="libgazebo_ros_camera.so">
-                <frame_name>camera_link_optical</frame_name>
-            </plugin>
-        </sensor>
-    </gazebo>
-    <joint name="camera2_joint" type="fixed">
-        <parent link="chassis"/>
-        <child link="camera2_link"/>
-        <origin xyz="0.32 -0.1400242 0.25" rpy="0 0 0"/>
-    </joint>
-    <link name="camera2_link">
-        <visual>
-            <geometry>
-                <box size="0.010 0.03 0.03"/>
-            </geometry>
-            <material name="red"/>
-        </visual>
-    </link>
-    <joint name="camera2_optical_joint" type="fixed">
-        <parent link="camera2_link"/>
-        <child link="camera2_link_optical"/>
-        <origin xyz="0 0 0" rpy="${-pi/2} 0 ${-pi/2}"/>
-    </joint>
-    <link name="camera2_link_optical"></link>
-    <gazebo reference="camera2_link">
-        <material>Gazebo/Red</material>
-        <sensor name="camera2" type="camera">
-            <pose> 0 0 0 0 0 0 </pose>
-            <visualize>true</visualize>
-            <update_rate>10</update_rate>
-            <camera>
-                <horizontal_fov>1.089</horizontal_fov>
-                <image>
-                    <format>R8G8B8</format>
-                    <width>640</width>
-                    <height>480</height>
-                </image>
-                <clip>
-                    <near>0.05</near>
-                    <far>8.0</far>
-                </clip>
-            </camera>
-            <plugin name="camera2_controller" filename="libgazebo_ros_camera.so">
-                <frame_name>camera2_link_optical</frame_name>
-            </plugin>
-        </sensor>
-    </gazebo>
+<robot xmlns:xacro="http://www.ros.org/wiki/xacro">
+  <!-- Camera 1 -->
+  <joint name="camera_joint" type="fixed">
+    <parent link="base_link"/> <!-- Changed parent to base_link -->
+    <child link="camera_link"/>
+    <origin xyz="0.15 0.14 0.25" rpy="0 0 0"/> <!-- Adjusted position -->
+  </joint>
+  <link name="camera_link">
+    <visual>
+      <geometry><box size="0.010 0.03 0.03"/></geometry>
+      <material name="red"/>
+    </visual>
+  </link>
+  <joint name="camera_optical_joint" type="fixed">
+    <parent link="camera_link"/>
+    <child link="camera_link_optical"/>
+    <origin xyz="0 0 0" rpy="${-M_PI/2} 0 ${-M_PI/2}"/>
+  </joint>
+  <link name="camera_link_optical"/>
+  <!-- Camera 2 -->
+  <joint name="camera2_joint" type="fixed">
+    <parent link="base_link"/> <!-- Changed parent to base_link -->
+    <child link="camera2_link"/>
+    <origin xyz="0.15 -0.14 0.25" rpy="0 0 0"/> <!-- Adjusted position -->
+  </joint>
+  <link name="camera2_link">
+    <visual>
+      <geometry><box size="0.010 0.03 0.03"/></geometry>
+      <material name="red"/>
+    </visual>
+  </link>
+  <joint name="camera2_optical_joint" type="fixed">
+    <parent link="camera2_link"/>
+    <child link="camera2_link_optical"/>
+    <origin xyz="0 0 0" rpy="${-M_PI/2} 0 ${-M_PI/2}"/>
+  </joint>
+  <link name="camera2_link_optical"/>
+  <!-- Gazebo Sensors -->
+  <gazebo reference="camera_link">
+    <material>Gazebo/Red</material>
+    <sensor name="camera" type="camera">
+      <pose>0 0 0 0 0 0</pose>
+      <update_rate>10</update_rate>
+      <camera>
+        <horizontal_fov>1.089</horizontal_fov>
+        <image><width>640</width><height>480</height></image>
+        <clip><near>0.05</near><far>8.0</far></clip>
+      </camera>
+      <plugin name="camera_controller" filename="libgazebo_ros_camera.so">
+        <frame_name>camera_link_optical</frame_name>
+      </plugin>
+    </sensor>
+  </gazebo>
+  <gazebo reference="camera2_link">
+    <material>Gazebo/Red</material>
+    <sensor name="camera2" type="camera">
+      <pose>0 0 0 0 0 0</pose>
+      <update_rate>10</update_rate>
+      <camera>
+        <horizontal_fov>1.089</horizontal_fov>
+        <image><width>640</width><height>480</height></image>
+        <clip><near>0.05</near><far>8.0</far></clip>
+      </camera>
+      <plugin name="camera2_controller" filename="libgazebo_ros_camera.so">
+        <frame_name>camera2_link_optical</frame_name>
+      </plugin>
+    </sensor>
+  </gazebo>
 </robot>

File: src/sec_bot/description/gazebo_control.xacro (robot description, xacro)
@@ -2,15 +2,16 @@
 <robot xmlns:xacro="http://www.ros.org/wiki/xacro">
   <gazebo>
-    <plugin name="gazebo_ros_control" filename="libgazebo_ros_control.so"/> <!-- loads Gazebo control -->
-    <plugin name="diff_drive" filename="libgazebo_ros_diff_drive.so"> <!-- differential drive plugin -->
-      <update_rate>50</update_rate> <!-- sets simulation update rate -->
-      <left_joint>left_front_wheel_joint left_back_wheel_joint</left_joint> <!-- left wheels -->
-      <right_joint>right_front_wheel_joint right_back_wheel_joint</right_joint> <!-- right wheels -->
-      <wheel_separation>0.35</wheel_separation> <!-- distance between wheels -->
-      <wheel_diameter>0.08</wheel_diameter> <!-- wheel size -->
-      <max_wheel_torque>5</max_wheel_torque> <!-- sets max torque -->
-      <max_wheel_acceleration>3</max_wheel_acceleration> <!-- Max acceleration -->
-      <odometry_frame>odom</odometry_frame> <!-- sses 'odom' frame -->
-      <robot_base_frame>base_footprint</robot_base_frame> <!-- uses base footprint -->
+    <plugin name="gazebo_ros_control" filename="libgazebo_ros_control.so"/>
+    <!-- Differential Drive Plugin (UPDATED FOR FOUR WHEELS!!!) -->
+    <plugin name="diff_drive" filename="libgazebo_ros_diff_drive.so">
+      <update_rate>50</update_rate>
+      <!-- Use only 1 joint per side (front wheels as representatives) -->
+      <left_joint>left_front_wheel_joint</left_joint>
+      <right_joint>right_front_wheel_joint</right_joint>
+      <wheel_separation>0.35</wheel_separation>
+      <wheel_diameter>0.08</wheel_diameter>
+      <max_wheel_torque>5</max_wheel_torque>
+      <odometry_frame>odom</odometry_frame>
+      <robot_base_frame>base_footprint</robot_base_frame>
     </plugin>
   </gazebo>

File: src/sec_bot/description/robot_core.xacro (robot description, xacro)
@@ -3,14 +3,14 @@
   <!-- Includes -->
   <xacro:include filename="inertial_macros.xacro"/>
-  <xacro:include filename="gazebo_control.xacro"/>
   <!-- Parameters -->
   <xacro:property name="M_PI" value="3.1415926535897931" />
-  <xacro:property name="left_back_wheel_pos" value="-0.02 0.175 0"/>
-  <xacro:property name="right_back_wheel_pos" value="-0.02 -0.175 0"/>
-  <xacro:property name="left_front_wheel_pos" value="0.2 0.175 0"/>
-  <xacro:property name="right_front_wheel_pos" value="0.2 -0.175 0"/>
+  <xacro:property name="left_back_wheel_pos" value="-0.15 0.15 0"/>
+  <xacro:property name="right_back_wheel_pos" value="-0.15 -0.15 0"/>
+  <xacro:property name="left_front_wheel_pos" value="0.15 0.15 0"/>
+  <xacro:property name="right_front_wheel_pos" value="0.15 -0.15 0"/>
   <!-- Materials -->
   <material name="white"><color rgba="1 1 1 1"/></material>
   <material name="blue"><color rgba="0.2 0.2 1 1"/></material>
+  <material name="red"><color rgba="1 0 0 1"/></material> <!-- Added -->
   <!-- Base Structure -->
   <link name="base_footprint"/>
@@ -27,21 +27,21 @@
     <origin xyz="-0.1 0 0"/>
   </joint>
-<link name="chassis">
-  <visual>
-    <geometry><box size="0.3 0.3 0.25"/></geometry>
-    <material name="white"/>
-  </visual>
-  <collision>
-    <geometry><box size="0.3 0.3 0.25"/></geometry>
-  </collision>
-  <xacro:inertial_box
-    mass="0.5"
-    x="0.3"
-    y="0.3"
-    z="0.25"
-    origin_xyz='0 0 0'
-    origin_rpy='0 0 0'
-  />
-</link>
+  <link name="chassis">
+    <visual>
+      <geometry><box size="0.3 0.3 0.25"/></geometry>
+      <material name="white"/>
+    </visual>
+    <collision>
+      <geometry><box size="0.3 0.3 0.25"/></geometry>
+    </collision>
+    <xacro:inertial_box
+      mass="0.5"
+      x="0.3"
+      y="0.3"
+      z="0.25"
+      origin_xyz='0 0 0'
+      origin_rpy='0 0 0'
+    />
+  </link>
   <!-- Wheels & Transmissions -->
   <xacro:macro name="full_wheel" params="name parent origin rpy axis">
@@ -74,10 +74,10 @@
   <!-- Instantiate Wheels -->
   <xacro:full_wheel name="left_back_wheel" parent="base_link"
-                    origin="${left_back_wheel_pos}" rpy="${-(M_PI/2)} 0 0" axis="0 0 1"/>
+                    origin="${left_back_wheel_pos}" rpy="${-(M_PI/2)} 0 0" axis="0 1 0"/>
   <xacro:full_wheel name="right_back_wheel" parent="base_link"
-                    origin="${right_back_wheel_pos}" rpy="${M_PI/2} 0 0" axis="0 0 -1"/>
+                    origin="${right_back_wheel_pos}" rpy="${M_PI/2} 0 0" axis="0 1 0"/>
   <xacro:full_wheel name="left_front_wheel" parent="base_link"
-                    origin="${left_front_wheel_pos}" rpy="${-(M_PI/2)} 0 0" axis="0 0 1"/>
+                    origin="${left_front_wheel_pos}" rpy="${-(M_PI/2)} 0 0" axis="0 1 0"/>
   <xacro:full_wheel name="right_front_wheel" parent="base_link"
-                    origin="${right_front_wheel_pos}" rpy="${M_PI/2} 0 0" axis="0 0 -1"/>
+                    origin="${right_front_wheel_pos}" rpy="${M_PI/2} 0 0" axis="0 1 0"/>
 </robot>

File: src/sec_bot/description/ros2_control.xacro (robot description, xacro)
@@ -1,62 +1,32 @@
 <?xml version="1.0"?>
 <robot xmlns:xacro="http://www.ros.org/wiki/xacro">
-    <xacro:unless value="$(arg sim_mode)">
-        <ros2_control name="RealRobot" type="system">
-            <hardware>
-                <plugin>diffdrive_arduino/DiffDriveArduino</plugin>
-                <param name="left_wheel_name">left_wheel_joint</param>
-                <param name="right_wheel_name">right_wheel_joint</param>
-                <param name="loop_rate">30</param>
-                <param name="device">/dev/ttyUSB0</param>
-                <param name="baud_rate">57600</param>
-                <param name="timeout">1000</param>
-                <param name="enc_counts_per_rev">3436</param>
-            </hardware>
-            <joint name="left_wheel_joint">
-                <command_interface name="velocity">
-                    <param name="min">-10</param>
-                    <param name="max">10</param>
-                </command_interface>
-                <state_interface name="velocity"/>
-                <state_interface name="position"/>
-            </joint>
-            <joint name="right_wheel_joint">
-                <command_interface name="velocity">
-                    <param name="min">-10</param>
-                    <param name="max">10</param>
-                </command_interface>
-                <state_interface name="velocity"/>
-                <state_interface name="position"/>
-            </joint>
-        </ros2_control>
-    </xacro:unless>
-    <xacro:if value="$(arg sim_mode)">
-        <ros2_control name="GazeboSystem" type="system">
-            <hardware>
-                <plugin>gazebo_ros2_control/GazeboSystem</plugin>
-            </hardware>
-            <joint name="left_wheel_joint">
-                <command_interface name="velocity">
-                    <param name="min">-10</param>
-                    <param name="max">10</param>
-                </command_interface>
-                <state_interface name="velocity"/>
-                <state_interface name="position"/>
-            </joint>
-            <joint name="right_wheel_joint">
-                <command_interface name="velocity">
-                    <param name="min">-10</param>
-                    <param name="max">10</param>
-                </command_interface>
-                <state_interface name="velocity"/>
-                <state_interface name="position"/>
-            </joint>
-        </ros2_control>
-    </xacro:if>
-    <gazebo>
-        <plugin name="gazebo_ros2_control" filename="libgazebo_ros2_control.so">
-            <parameters>$(find articubot_one)/config/my_controllers.yaml</parameters>
-            <parameters>$(find articubot_one)/config/gaz_ros2_ctl_use_sim.yaml</parameters>
-        </plugin>
-    </gazebo>
+  <xacro:if value="$(arg sim_mode)">
+    <ros2_control name="GazeboSystem" type="system">
+      <hardware>
+        <plugin>gazebo_ros2_control/GazeboSystem</plugin>
+      </hardware>
+      <!-- Include all four wheel joints -->
+      <joint name="left_front_wheel_joint">
+        <command_interface name="velocity"/>
+        <state_interface name="velocity"/>
+      </joint>
+      <joint name="left_back_wheel_joint">
+        <command_interface name="velocity"/>
+        <state_interface name="velocity"/>
+      </joint>
+      <joint name="right_front_wheel_joint">
+        <command_interface name="velocity"/>
+        <state_interface name="velocity"/>
+      </joint>
+      <joint name="right_back_wheel_joint">
+        <command_interface name="velocity"/>
+        <state_interface name="velocity"/>
+      </joint>
+    </ros2_control>
+  </xacro:if>
+  <gazebo>
+    <plugin name="gazebo_ros2_control" filename="libgazebo_ros2_control.so">
+      <parameters>$(find articubot_one)/config/my_controllers.yaml</parameters>
+    </plugin>
+  </gazebo>
 </robot>
