Commit message: please work

File: src/sec_bot/description/camera.xacro (robot description, xacro)
@@ -1,7 +1,4 @@
 <?xml version="1.0"?>
 <robot xmlns:xacro="http://www.ros.org/wiki/xacro" >
-  <material name="red">
-    <color rgba="1 0 0 1"/>
-  </material>
     <joint name="camera_joint" type="fixed">
         <parent link="chassis"/>

File: src/sec_bot/description/gazebo_control.xacro (robot description, xacro)
@@ -1,9 +1,20 @@
 <?xml version="1.0"?>
-<robot xmlns:xacro="http://www.ros.org/wiki/xacro">
+<robot xmlns:xacro="http://www.ros.org/wiki/xacro"  name="robot">
   <gazebo>
-    <!-- ROS 2 control Gazebo plugin -->
-    <plugin name="gazebo_ros2_control" filename="libgazebo_ros2_control.so">
-      <!-- Path to controller configuration YAML -->
-      <parameters>$(find sec_bot)/config/controllers.yaml</parameters>
+    <plugin name="diff_drive" filename="libgazebo_ros_diff_drive.so">
+      <!-- FIX: ensured all 4 wheels are included -->
+      <left_joint> left_front_wheel_joint </left_joint>
+      <left_joint> left_back_wheel_joint </left_joint>
+      <right_joint> right_front_wheel_joint </right_joint>
+      <right_joint> right_back_wheel_joint </right_joint>
+      <wheel_separation>0.2800484</wheel_separation>
+      <wheel_diameter>0.1651</wheel_diameter>
+      <max_wheel_torque>200</max_wheel_torque>
+      <max_wheel_acceleration>10</max_wheel_acceleration>
+      <odometry_frame>odom</odometry_frame>
+      <robot_base_frame>base_link</robot_base_frame>
+      <publish_odom>true</publish_odom>
+      <publish_odom_tf>true</publish_odom_tf>
+      <publish_wheel_tf>true</publish_wheel_tf>
     </plugin>
   </gazebo>

File: src/sec_bot/description/ros2_control.xacro (robot description, xacro)
@@ -1,87 +1,69 @@
 <?xml version="1.0"?>
 <robot xmlns:xacro="http://www.ros.org/wiki/xacro">
-    <xacro:unless value="$(arg sim_mode)">
-        <ros2_control name="RealRobot" type="system">
-            <hardware>
-                <plugin>diffdrive_arduino/DiffDriveArduino</plugin>
-                <param name="left_wheel_name">left_front_wheel_joint left_back_wheel_joint</param>
-                <param name="right_wheel_name">right_front_wheel_joint right_back_wheel_joint</param>
-                <param name="loop_rate">30</param>
-                <param name="device">/dev/ttyUSB0</param>
-                <param name="baud_rate">57600</param>
-                <param name="timeout">1000</param>
-                <param name="enc_counts_per_rev">3436</param>
-            </hardware>
-            <!-- Front Left Wheel -->
-            <joint name="left_front_wheel_joint">
-                <command_interface name="velocity">
-                    <param name="min">-10</param>
-                    <param name="max">10</param>
-                </command_interface>
-                <state_interface name="velocity"/>
-                <state_interface name="position"/>
-            </joint>
-            <!-- Back Left Wheel -->
-            <joint name="left_back_wheel_joint">
-                <command_interface name="velocity">
-                    <param name="min">-10</param>
-                    <param name="max">10</param>
-                </command_interface>
-                <state_interface name="velocity"/>
-                <state_interface name="position"/>
-            </joint>
-            <!-- Front Right Wheel -->
-            <joint name="right_front_wheel_joint">
-                <command_interface name="velocity">
-                    <param name="min">-10</param>
-                    <param name="max">10</param>
-                </command_interface>
-                <state_interface name="velocity"/>
-                <state_interface name="position"/>
-            </joint>
-            <!-- Back Right Wheel -->
-            <joint name="right_back_wheel_joint">
-                <command_interface name="velocity">
-                    <param name="min">-10</param>
-                    <param name="max">10</param>
-                </command_interface>
-                <state_interface name="velocity"/>
-                <state_interface name="position"/>
-            </joint>
-        </ros2_control>
-    </xacro:unless>
-    <xacro:if value="$(arg sim_mode)">
-        <ros2_control name="GazeboSystem" type="system">
-            <hardware>
-                <plugin>gazebo_ros2_control/GazeboSystem</plugin>
-            </hardware>
-            <!-- Identical joint declarations for simulation -->
-            <joint name="left_front_wheel_joint">
-                <command_interface name="velocity"/>
-                <state_interface name="velocity"/>
-                <state_interface name="position"/>
-            </joint>
-            <joint name="left_back_wheel_joint">
-                <command_interface name="velocity"/>
-                <state_interface name="velocity"/>
-                <state_interface name="position"/>
-            </joint>
-            <joint name="right_front_wheel_joint">
-                <command_interface name="velocity"/>
-                <state_interface name="velocity"/>
-                <state_interface name="position"/>
-            </joint>
-            <joint name="right_back_wheel_joint">
-                <command_interface name="velocity"/>
-                <state_interface name="velocity"/>
-                <state_interface name="position"/>
-            </joint>
-        </ros2_control>
-    </xacro:if>
-    <gazebo>
-        <plugin name="gazebo_ros2_control" filename="libgazebo_ros2_control.so">
-            <parameters>$(find articubot_one)/config/my_controllers.yaml</parameters>
-            <parameters>$(find articubot_one)/config/gaz_ros2_ctl_use_sim.yaml</parameters>
-        </plugin>
-    </gazebo>
+  <!-- REAL HARDWARE CONFIG (Arduino) -->
+  <xacro:unless value="$(arg sim_mode)">
+    <ros2_control name="RealRobot" type="system">
+      <hardware>
+        <plugin>diffdrive_arduino/DiffDriveArduino</plugin>
+        <param name="left_wheel_name">left_front_wheel_joint</param>
+        <param name="right_wheel_name">right_front_wheel_joint</param>
+        <param name="loop_rate">30</param>
+        <param name="device">/dev/ttyUSB0</param>
+        <param name="baud_rate">57600</param>
+        <param name="timeout">1000</param>
+        <param name="enc_counts_per_rev">3436</param>
+      </hardware>
+      <joint name="left_front_wheel_joint">
+        <command_interface name="velocity">
+          <param name="min">-10</param>
+          <param name="max">10</param>
+        </command_interface>
+        <state_interface name="velocity"/>
+        <state_interface name="position"/>
+      </joint>
+      <joint name="right_front_wheel_joint">
+        <command_interface name="velocity">
+          <param name="min">-10</param>
+          <param name="max">10</param>
+        </command_interface>
+        <state_interface name="velocity"/>
+        <state_interface name="position"/>
+      </joint>
+    </ros2_control>
+  </xacro:unless>
+  <!-- GAZEBO SIMULATION CONFIG -->
+  <xacro:if value="$(arg sim_mode)">
+    <ros2_control name="GazeboSystem" type="system">
+      <hardware>
+        <plugin>gazebo_ros2_control/GazeboSystem</plugin>
+      </hardware>
+      <!-- All 4 wheel joints -->
+      <joint name="left_front_wheel_joint">
+        <command_interface name="velocity"/>
+        <state_interface name="velocity"/>
+        <state_interface name="position"/>
+      </joint>
+      <joint name="left_back_wheel_joint">
+        <command_interface name="velocity"/>
+        <state_interface name="velocity"/>
+        <state_interface name="position"/>
+      </joint>
+      <joint name="right_front_wheel_joint">
+        <command_interface name="velocity"/>
+        <state_interface name="velocity"/>
+        <state_interface name="position"/>
+      </joint>
+      <joint name="right_back_wheel_joint">
+        <command_interface name="velocity"/>
+        <state_interface name="velocity"/>
+        <state_interface name="position"/>
+      </joint>
+    </ros2_control>
+  </xacro:if>
+  <gazebo>
+    <plugin name="gazebo_ros2_control" filename="libgazebo_ros2_control.so">
+      <!-- Single parameters file for controllers -->
+      <parameters>$(find articubot_one)/config/my_controllers.yaml</parameters>
+    </plugin>
+  </gazebo>
 </robot>

Commit message: Revert "please work"
This reverts commit 8bbb435bd9fc42d32b77e317ce1eb027efbf3fb3.

File: src/sec_bot/description/camera.xacro (robot description, xacro)
@@ -1,4 +1,7 @@
 <?xml version="1.0"?>
 <robot xmlns:xacro="http://www.ros.org/wiki/xacro" >
+  <material name="red">
+    <color rgba="1 0 0 1"/>
+  </material>
     <joint name="camera_joint" type="fixed">
         <parent link="chassis"/>

File: src/sec_bot/description/gazebo_control.xacro (robot description, xacro)
@@ -1,20 +1,9 @@
 <?xml version="1.0"?>
-<robot xmlns:xacro="http://www.ros.org/wiki/xacro"  name="robot">
+<robot xmlns:xacro="http://www.ros.org/wiki/xacro">
   <gazebo>
-    <plugin name="diff_drive" filename="libgazebo_ros_diff_drive.so">
-      <!-- FIX: ensured all 4 wheels are included -->
-      <left_joint> left_front_wheel_joint </left_joint>
-      <left_joint> left_back_wheel_joint </left_joint>
-      <right_joint> right_front_wheel_joint </right_joint>
-      <right_joint> right_back_wheel_joint </right_joint>
-      <wheel_separation>0.2800484</wheel_separation>
-      <wheel_diameter>0.1651</wheel_diameter>
-      <max_wheel_torque>200</max_wheel_torque>
-      <max_wheel_acceleration>10</max_wheel_acceleration>
-      <odometry_frame>odom</odometry_frame>
-      <robot_base_frame>base_link</robot_base_frame>
-      <publish_odom>true</publish_odom>
-      <publish_odom_tf>true</publish_odom_tf>
-      <publish_wheel_tf>true</publish_wheel_tf>
+    <!-- ROS 2 control Gazebo plugin -->
+    <plugin name="gazebo_ros2_control" filename="libgazebo_ros2_control.so">
+      <!-- Path to controller configuration YAML -->
+      <parameters>$(find sec_bot)/config/controllers.yaml</parameters>
     </plugin>
   </gazebo>

File: src/sec_bot/description/ros2_control.xacro (robot description, xacro)
@@ -1,69 +1,87 @@
 <?xml version="1.0"?>
 <robot xmlns:xacro="http://www.ros.org/wiki/xacro">
-  <!-- REAL HARDWARE CONFIG (Arduino) -->
-  <xacro:unless value="$(arg sim_mode)">
-    <ros2_control name="RealRobot" type="system">
-      <hardware>
-        <plugin>diffdrive_arduino/DiffDriveArduino</plugin>
-        <param name="left_wheel_name">left_front_wheel_joint</param>
-        <param name="right_wheel_name">right_front_wheel_joint</param>
-        <param name="loop_rate">30</param>
-        <param name="device">/dev/ttyUSB0</param>
-        <param name="baud_rate">57600</param>
-        <param name="timeout">1000</param>
-        <param name="enc_counts_per_rev">3436</param>
-      </hardware>
-      <joint name="left_front_wheel_joint">
-        <command_interface name="velocity">
-          <param name="min">-10</param>
-          <param name="max">10</param>
-        </command_interface>
-        <state_interface name="velocity"/>
-        <state_interface name="position"/>
-      </joint>
-      <joint name="right_front_wheel_joint">
-        <command_interface name="velocity">
-          <param name="min">-10</param>
-          <param name="max">10</param>
-        </command_interface>
-        <state_interface name="velocity"/>
-        <state_interface name="position"/>
-      </joint>
-    </ros2_control>
-  </xacro:unless>
-  <!-- GAZEBO SIMULATION CONFIG -->
-  <xacro:if value="$(arg sim_mode)">
-    <ros2_control name="GazeboSystem" type="system">
-      <hardware>
-        <plugin>gazebo_ros2_control/GazeboSystem</plugin>
-      </hardware>
-      <!-- All 4 wheel joints -->
-      <joint name="left_front_wheel_joint">
-        <command_interface name="velocity"/>
-        <state_interface name="velocity"/>
-        <state_interface name="position"/>
-      </joint>
-      <joint name="left_back_wheel_joint">
-        <command_interface name="velocity"/>
-        <state_interface name="velocity"/>
-        <state_interface name="position"/>
-      </joint>
-      <joint name="right_front_wheel_joint">
-        <command_interface name="velocity"/>
-        <state_interface name="velocity"/>
-        <state_interface name="position"/>
-      </joint>
-      <joint name="right_back_wheel_joint">
-        <command_interface name="velocity"/>
-        <state_interface name="velocity"/>
-        <state_interface name="position"/>
-      </joint>
-    </ros2_control>
-  </xacro:if>
-  <gazebo>
-    <plugin name="gazebo_ros2_control" filename="libgazebo_ros2_control.so">
-      <!-- Single parameters file for controllers -->
-      <parameters>$(find articubot_one)/config/my_controllers.yaml</parameters>
-    </plugin>
-  </gazebo>
+    <xacro:unless value="$(arg sim_mode)">
+        <ros2_control name="RealRobot" type="system">
+            <hardware>
+                <plugin>diffdrive_arduino/DiffDriveArduino</plugin>
+                <param name="left_wheel_name">left_front_wheel_joint left_back_wheel_joint</param>
+                <param name="right_wheel_name">right_front_wheel_joint right_back_wheel_joint</param>
+                <param name="loop_rate">30</param>
+                <param name="device">/dev/ttyUSB0</param>
+                <param name="baud_rate">57600</param>
+                <param name="timeout">1000</param>
+                <param name="enc_counts_per_rev">3436</param>
+            </hardware>
+            <!-- Front Left Wheel -->
+            <joint name="left_front_wheel_joint">
+                <command_interface name="velocity">
+                    <param name="min">-10</param>
+                    <param name="max">10</param>
+                </command_interface>
+                <state_interface name="velocity"/>
+                <state_interface name="position"/>
+            </joint>
+            <!-- Back Left Wheel -->
+            <joint name="left_back_wheel_joint">
+                <command_interface name="velocity">
+                    <param name="min">-10</param>
+                    <param name="max">10</param>
+                </command_interface>
+                <state_interface name="velocity"/>
+                <state_interface name="position"/>
+            </joint>
+            <!-- Front Right Wheel -->
+            <joint name="right_front_wheel_joint">
+                <command_interface name="velocity">
+                    <param name="min">-10</param>
+                    <param name="max">10</param>
+                </command_interface>
+                <state_interface name="velocity"/>
+                <state_interface name="position"/>
+            </joint>
+            <!-- Back Right Wheel -->
+            <joint name="right_back_wheel_joint">
+                <command_interface name="velocity">
+                    <param name="min">-10</param>
+                    <param name="max">10</param>
+                </command_interface>
+                <state_interface name="velocity"/>
+                <state_interface name="position"/>
+            </joint>
+        </ros2_control>
+    </xacro:unless>
+    <xacro:if value="$(arg sim_mode)">
+        <ros2_control name="GazeboSystem" type="system">
+            <hardware>
+                <plugin>gazebo_ros2_control/GazeboSystem</plugin>
+            </hardware>
+            <!-- Identical joint declarations for simulation -->
+            <joint name="left_front_wheel_joint">
+                <command_interface name="velocity"/>
+                <state_interface name="velocity"/>
+                <state_interface name="position"/>
+            </joint>
+            <joint name="left_back_wheel_joint">
+                <command_interface name="velocity"/>
+                <state_interface name="velocity"/>
+                <state_interface name="position"/>
+            </joint>
+            <joint name="right_front_wheel_joint">
+                <command_interface name="velocity"/>
+                <state_interface name="velocity"/>
+                <state_interface name="position"/>
+            </joint>
+            <joint name="right_back_wheel_joint">
+                <command_interface name="velocity"/>
+                <state_interface name="velocity"/>
+                <state_interface name="position"/>
+            </joint>
+        </ros2_control>
+    </xacro:if>
+    <gazebo>
+        <plugin name="gazebo_ros2_control" filename="libgazebo_ros2_control.so">
+            <parameters>$(find articubot_one)/config/my_controllers.yaml</parameters>
+            <parameters>$(find articubot_one)/config/gaz_ros2_ctl_use_sim.yaml</parameters>
+        </plugin>
+    </gazebo>
 </robot>

Commit message: lets try the changes to gazebo_control

File: src/sec_bot/description/camera.xacro (robot description, xacro)
@@ -1,7 +1,7 @@
 <?xml version="1.0"?>
 <robot xmlns:xacro="http://www.ros.org/wiki/xacro" >
-  <material name="red">
-    <color rgba="1 0 0 1"/>
-  </material>
+    <material name="red">
+      <color rgba="1 0 0 1"/>
+    </material>
     <joint name="camera_joint" type="fixed">
         <parent link="chassis"/>

File: src/sec_bot/description/gazebo_control.xacro (robot description, xacro)
@@ -5,5 +5,33 @@
     <plugin name="gazebo_ros2_control" filename="libgazebo_ros2_control.so">
       <!-- Path to controller configuration YAML -->
-      <parameters>$(find sec_bot)/config/controllers.yaml</parameters>
+      <!-- <parameters>$(find sec_bot)/config/controllers.yaml</parameters> -->
+      <!-- 2 wheels per side -->
+      <num_wheel_pairs>2</num_wheel_pairs>
+      <!-- Left Wheels -->
+      <left_joint>
+        left_front_wheel_joint
+      </left_joint>
+      <left_joint>
+        left_back_wheel_joint
+      </left_joint>
+      <!-- Right Wheels -->
+      <right_joint>
+        right_front_wheel_joint
+      </right_joint>
+      <right_joint>
+        right_back_wheel_joint
+      </right_joint>
+      <!-- Wheel Definitions -->
+      <wheel_seperation>0.2800484</wheel_seperation>
+      <wheel_diameter>0.1651</wheel_diameter>
+      <!-- Limits -->
+      <max_wheel_torque>200</max_wheel_torque>
+      <max_wheel_acceleration>10</max_wheel_acceleration>
+      <!-- Output -->
+      <odometry_frame>odom</odometry_frame>
+      <robot_base_frame>base_link</robot_base_frame>
+      <publish_odom>true</publish_odom>
+      <publish_odom_tf>true</publish_odom_tf>
+      <publish_wheel_tf>true</publish_wheel_tf>
     </plugin>
   </gazebo>

Commit message: added camera_red

File: src/sec_bot/description/camera.xacro (robot description, xacro)
@@ -1,5 +1,5 @@
 <?xml version="1.0"?>
 <robot xmlns:xacro="http://www.ros.org/wiki/xacro" >
-    <material name="red">
+    <material name="camera_red">
       <color rgba="1 0 0 1"/>
     </material>
@@ -14,5 +14,5 @@
                 <box size="0.010 0.03 0.03"/>
             </geometry>
-            <material name="red"/>
+            <material name="camera_red"/>
         </visual>
     </link>
@@ -56,5 +56,5 @@
                 <box size="0.010 0.03 0.03"/>
             </geometry>
-            <material name="red"/>
+            <material name="camera_red"/>
         </visual>
     </link>
