Commit message: rweywgerwegr

File: src/sec_bot/description/camera.xacro (robot description, xacro)
@@ -4,8 +4,9 @@
       <color rgba="1 0 0 1"/>
     </material>
+    <!-- Left Camera -->
     <joint name="camera_joint" type="fixed">
         <parent link="chassis"/>
         <child link="camera_link"/>
-        <origin xyz="0.32 0.1400242 0.25" rpy="0 0 0"/>
+        <origin xyz="0.12 0.12 0.25" rpy="0 0 0"/>
     </joint>
     <link name="camera_link">
@@ -16,4 +17,13 @@
             <material name="camera_red"/>
         </visual>
+        <collision>
+            <geometry>
+                <box size="0.010 0.03 0.03"/>
+            </geometry>
+        </collision>
+        <inertial>
+            <mass value="0.05"/>
+            <inertia ixx="0.0001" ixy="0" ixz="0" iyy="0.0001" iyz="0" izz="0.0001"/>
+        </inertial>
     </link>
     <joint name="camera_optical_joint" type="fixed">
@@ -23,31 +33,9 @@
     </joint>
     <link name="camera_link_optical"></link>
-    <gazebo reference="camera_link">
-        <material>Gazebo/Red</material>
-        <sensor name="camera" type="camera">
-            <pose> 0 0 0 0 0 0 </pose>
-            <visualize>true</visualize>
-            <update_rate>10</update_rate>
-            <camera>
-                <horizontal_fov>1.089</horizontal_fov>
-                <image>
-                    <format>R8G8B8</format>
-                    <width>640</width>
-                    <height>480</height>
-                </image>
-                <clip>
-                    <near>0.05</near>
-                    <far>8.0</far>
-                </clip>
-            </camera>
-            <plugin name="camera_controller" filename="libgazebo_ros_camera.so">
-                <frame_name>camera_link_optical</frame_name>
-            </plugin>
-        </sensor>
-    </gazebo>
+    <!-- Right Camera -->
     <joint name="camera2_joint" type="fixed">
         <parent link="chassis"/>
         <child link="camera2_link"/>
-        <origin xyz="0.32 -0.1400242 0.25" rpy="0 0 0"/>
+        <origin xyz="0.12 -0.12 0.25" rpy="0 0 0"/>
     </joint>
     <link name="camera2_link">
@@ -58,4 +46,13 @@
             <material name="camera_red"/>
         </visual>
+        <collision>
+            <geometry>
+                <box size="0.010 0.03 0.03"/>
+            </geometry>
+        </collision>
+        <inertial>
+            <mass value="0.05"/>
+            <inertia ixx="0.0001" ixy="0" ixz="0" iyy="0.0001" iyz="0" izz="0.0001"/>
+        </inertial>
     </link>
     <joint name="camera2_optical_joint" type="fixed">
@@ -65,26 +62,3 @@
     </joint>
     <link name="camera2_link_optical"></link>
-    <gazebo reference="camera2_link">
-        <material>Gazebo/Red</material>
-        <sensor name="camera2" type="camera">
-            <pose> 0 0 0 0 0 0 </pose>
-            <visualize>true</visualize>
-            <update_rate>10</update_rate>
-            <camera>
-                <horizontal_fov>1.089</horizontal_fov>
-                <image>
-                    <format>R8G8B8</format>
-                    <width>640</width>
-                    <height>480</height>
-                </image>
-                <clip>
-                    <near>0.05</near>
-                    <far>8.0</far>
-                </clip>
-            </camera>
-            <plugin name="camera2_controller" filename="libgazebo_ros_camera.so">
-                <frame_name>camera2_link_optical</frame_name>
-            </plugin>
-        </sensor>
-    </gazebo>
 </robot>

File: src/sec_bot/description/gazebo_control.xacro (robot description, xacro)
@@ -3,36 +3,5 @@
     <!-- Define PI if not already defined -->
     <xacro:property name="PI" value="3.1415926535897931" />
-    <material name="gazebo_red">
-      <color rgba="1 0 0 1"/>
-    </material>
-    <!-- Left Camera: Positioned on top-left corner of chassis -->
-    <joint name="camera_joint" type="fixed">
-        <parent link="chassis"/>
-        <child link="camera_link"/>
-        <origin xyz="0.12 0.12 0.25" rpy="0 0 0"/>  <!-- Moved to top-left of chassis -->
-    </joint>
-    <link name="camera_link">
-        <visual>
-            <geometry>
-                <box size="0.010 0.03 0.03"/>
-            </geometry>
-            <material name="gazebo_red"/>
-        </visual>
-        <collision>
-            <geometry>
-                <box size="0.010 0.03 0.03"/>
-            </geometry>
-        </collision>
-        <inertial>
-            <mass value="0.05"/>
-            <inertia ixx="0.0001" ixy="0" ixz="0" iyy="0.0001" iyz="0" izz="0.0001"/>
-        </inertial>
-    </link>
-    <joint name="camera_optical_joint" type="fixed">
-        <parent link="camera_link"/>
-        <child link="camera_link_optical"/>
-        <origin xyz="0 0 0" rpy="${-PI/2} 0 ${-PI/2}"/>
-    </joint>
-    <link name="camera_link_optical"></link>
+    <!-- Camera Gazebo Integration -->
     <gazebo reference="camera_link">
         <material>Gazebo/Red</material>
@@ -58,33 +27,4 @@
         </sensor>
     </gazebo>
-    <!-- Right Camera: Positioned on top-right corner of chassis -->
-    <joint name="camera2_joint" type="fixed">
-        <parent link="chassis"/>
-        <child link="camera2_link"/>
-        <origin xyz="0.12 -0.12 0.25" rpy="0 0 0"/>  <!-- Moved to top-right of chassis -->
-    </joint>
-    <link name="camera2_link">
-        <visual>
-            <geometry>
-                <box size="0.010 0.03 0.03"/>
-            </geometry>
-            <material name="gazebo_red"/>
-        </visual>
-        <collision>
-            <geometry>
-                <box size="0.010 0.03 0.03"/>
-            </geometry>
-        </collision>
-        <inertial>
-            <mass value="0.05"/>
-            <inertia ixx="0.0001" ixy="0" ixz="0" iyy="0.0001" iyz="0" izz="0.0001"/>
-        </inertial>
-    </link>
-    <joint name="camera2_optical_joint" type="fixed">
-        <parent link="camera2_link"/>
-        <child link="camera2_link_optical"/>
-        <origin xyz="0 0 0" rpy="${-PI/2} 0 ${-PI/2}"/>
-    </joint>
-    <link name="camera2_link_optical"></link>
     <gazebo reference="camera2_link">
         <material>Gazebo/Red</material>
@@ -110,3 +50,4 @@
         </sensor>
     </gazebo>
+    <!-- Add other Gazebo control plugins here -->
 </robot>
