Commit message: Finished up basic URDF to be modified later

File: src/sec_bot/description/robot_core.xacro (robot description, xacro)
@@ -2,5 +2,5 @@
 <robot xmlns:xacro="http://www.ros.org/wiki/xacro" >
     <xacro:include filename="inertial_macros.xacro"/>
-   <material name="white">
+    <material name="white">
         <color rgba="1 1 1 1" />
     </material>
@@ -13,7 +13,4 @@
     <material name="black">
         <color rgba="0 0 0 1"/>
-    </material>
-    <material name="red">
-        <color rgba="1 0 0 1"/>
     </material>
     <!-- BASE LINK -->
@@ -32,5 +29,5 @@
                 <box size="0.3 0.3 0.15"/>
             </geometry>
-            <material name="orange"/>
+            <material name="white"/>
         </visual>
         <collision>
@@ -39,47 +36,55 @@
                 <box size="0.3 0.3 0.15"/>
             </geometry>
-            <material name="orange"/>
         </collision>
+        <xacro:inertial_box mass="0.5" x="0.3" y="0.3" z="0.15">
+            <origin xyz="0.15 0 0.075" rpy="0 0 0"/>
+        </xacro:inertial_box>
     </link>
-        <!-- LEFT WHEEL LINK -->
-        <joint name ="left_wheel_joint" type="continuous">
-            <parent link="base_link"/>
-            <child link ="left_wheel"/>
-            <origin xyz="0 0.175 0" rpy="-${pi/2} 0 0"/>
-            <axis xyz="0 0 1"/>
-        </joint>
-        <link name="left_wheel">
-            <visual>
-                <geometry>
-                    <cylinder radius="0.05" length="0.04"/>
-                </geometry>
-                <material name = "blue"/>
-            </visual>
-            <collision>
-                <geometry>
-                    <cylinder radius="0.05" length="0.04"/>
-                </geometry>
-            </collision>
-        </link>
-        <!-- RIGHT WHEEL LINK -->
-        <joint name ="right_wheel_joint" type="continuous">
-            <parent link="base_link"/>
-            <child link ="right_wheel"/>
-            <origin xyz="0 0.175 0" rpy="-${pi/2} 0 0"/>
-            <axis xyz="0 0 -1"/>
-        </joint>
-        <link name="right_wheel">
-            <visual>
-                <geometry>
-                    <cylinder radius="0.05" length="0.04"/>
-                </geometry>
-                <material name = "blue"/>
-            </visual>
-            <collision>
-                <geometry>
-                    <cylinder radius="0.05" length="0.04"/>
-                </geometry>
-            </collision>
-        </link>
+    <!-- LEFT WHEEL LINK -->
+    <joint name="left_wheel_joint" type="continuous">
+        <parent link="base_link"/>
+        <child link="left_wheel"/>
+        <origin xyz="0 0.175 0" rpy="-${pi/2} 0 0" />
+        <axis xyz="0 0 1"/>
+    </joint>
+    <link name="left_wheel">
+        <visual>
+            <geometry>
+                <cylinder radius="0.05" length="0.04"/>
+            </geometry>
+            <material name="blue"/>
+        </visual>
+        <collision>
+            <geometry>
+                <cylinder radius="0.05" length="0.04"/>
+            </geometry>
+        </collision>
+        <xacro:inertial_cylinder mass="0.1" length="0.04" radius="0.05">
+            <origin xyz="0 0 0" rpy="0 0 0"/>
+        </xacro:inertial_cylinder>
+    </link>
+    <!-- RIGHT WHEEL LINK -->
+    <joint name="right_wheel_joint" type="continuous">
+        <parent link="base_link"/>
+        <child link="right_wheel"/>
+        <origin xyz="0 -0.175 0" rpy="${pi/2} 0 0" />
+        <axis xyz="0 0 -1"/>
+    </joint>
+    <link name="right_wheel">
+        <visual>
+            <geometry>
+                <cylinder radius="0.05" length="0.04"/>
+            </geometry>
+            <material name="blue"/>
+        </visual>
+        <collision>
+            <geometry>
+                <cylinder radius="0.05" length="0.04"/>
+            </geometry>
+        </collision>
+        <xacro:inertial_cylinder mass="0.1" length="0.04" radius="0.05">
+            <origin xyz="0 0 0" rpy="0 0 0"/>
+        </xacro:inertial_cylinder>
+    </link>
     <!-- CASTER WHEEL LINK -->
     <joint name="caster_wheel_joint" type="fixed">
@@ -91,5 +96,5 @@
         <visual>
             <geometry>
-                <sphere radius="$0.05"/>
+                <sphere radius="0.05"/>
             </geometry>
             <material name="black"/>
@@ -97,7 +102,10 @@
         <collision>
             <geometry>
-                <sphere radius="$0.05"/>
+                <sphere radius="0.05"/>
             </geometry>
         </collision>
+        <xacro:inertial_sphere mass="0.1" radius="0.05">
+            <origin xyz="0 0 0" rpy="0 0 0"/>
+        </xacro:inertial_sphere>
     </link>
 </robot>

Commit message: adjusted urdf

File: src/sec_bot/description/robot_core.xacro (robot description, xacro)
@@ -25,12 +25,12 @@
     <link name="chassis">
         <visual>
-            <origin xyz="0.15 0 0.075"/>
+            <origin xyz="0.19 0 0.125"/>
             <geometry>
-                <box size="0.3 0.3 0.15"/>
+                <box size="0.3 0.3 0.25"/>
             </geometry>
             <material name="white"/>
         </visual>
         <collision>
-            <origin xyz="0.15 0 0.075"/>
+            <origin xyz="0.19 0 0.125"/>
             <geometry>
                 <box size="0.3 0.3 0.15"/>
@@ -44,15 +44,15 @@
         <material>Gazebo/White</material>
     </gazebo>
-    <!-- LEFT WHEEL LINK -->
-    <joint name="left_wheel_joint" type="continuous">
+    <!-- LEFT BACK WHEEL LINK -->
+    <joint name="left_back_wheel_joint" type="continuous">
         <parent link="base_link"/>
-        <child link="left_wheel"/>
-        <origin xyz="0 0.175 0" rpy="-${pi/2} 0 0" />
+        <child link="left_back_wheel"/>
+        <origin xyz="-0.02 0.175 0" rpy="-${pi/2} 0 0" />
         <axis xyz="0 0 1"/>
     </joint>
-    <link name="left_wheel">
+    <link name="left_back_wheel">
         <visual>
             <geometry>
-                <cylinder radius="0.05" length="0.04"/>
+                <cylinder radius="0.04" length="0.04"/>
             </geometry>
             <material name="blue"/>
@@ -60,5 +60,5 @@
         <collision>
             <geometry>
-                <cylinder radius="0.05" length="0.04"/>
+                <cylinder radius="0.04" length="0.04"/>
             </geometry>
         </collision>
@@ -67,18 +67,18 @@
         </xacro:inertial_cylinder>
     </link>
-    <gazebo reference="left_wheel">
+    <gazebo reference="left_back_wheel">
         <material>Gazebo/Blue</material>
     </gazebo>
-    <!-- RIGHT WHEEL LINK -->
-    <joint name="right_wheel_joint" type="continuous">
+    <!-- RIGHT BACK WHEEL LINK -->
+    <joint name="right_back_wheel_joint" type="continuous">
         <parent link="base_link"/>
-        <child link="right_wheel"/>
-        <origin xyz="0 -0.175 0" rpy="${pi/2} 0 0" />
+        <child link="right_back_wheel"/>
+        <origin xyz="-0.02 -0.175 0" rpy="${pi/2} 0 0" />
         <axis xyz="0 0 -1"/>
     </joint>
-    <link name="right_wheel">
+    <link name="right_back_wheel">
         <visual>
             <geometry>
-                <cylinder radius="0.05" length="0.04"/>
+                <cylinder radius="0.04" length="0.04"/>
             </geometry>
             <material name="blue"/>
@@ -86,5 +86,5 @@
         <collision>
             <geometry>
-                <cylinder radius="0.05" length="0.04"/>
+                <cylinder radius="0.04" length="0.04"/>
             </geometry>
         </collision>
@@ -93,31 +93,58 @@
         </xacro:inertial_cylinder>
     </link>
-    <gazebo reference="right_wheel">
+    <gazebo reference="right_back_wheel">
         <material>Gazebo/Blue</material>
     </gazebo>
-    <!-- CASTER WHEEL LINK -->
-    <joint name="caster_wheel_joint" type="fixed">
-        <parent link="chassis"/>
-        <child link="caster_wheel"/>
-        <origin xyz="0.24 0 0"/>
+    <!-- LEFT FRONT WHEEL LINK -->
+    <joint name="left_front_wheel_joint" type="continuous">
+        <parent link="base_link"/>
+        <child link="left_front_wheel"/>
+        <origin xyz="0.2 0.175 0" rpy="-${pi/2} 0 0" />
+        <axis xyz="0 0 1"/>
     </joint>
-    <link name="caster_wheel">
+    <link name="left_front_wheel">
         <visual>
             <geometry>
-                <sphere radius="0.05"/>
+                <cylinder radius="0.04" length="0.04"/>
             </geometry>
-            <material name="black"/>
+            <material name="blue"/>
         </visual>
         <collision>
             <geometry>
-                <sphere radius="0.05"/>
+                <cylinder radius="0.04" length="0.04"/>
             </geometry>
         </collision>
-        <xacro:inertial_sphere mass="0.1" radius="0.05">
+        <xacro:inertial_cylinder mass="0.1" length="0.04" radius="0.05">
             <origin xyz="0 0 0" rpy="0 0 0"/>
-        </xacro:inertial_sphere>
+        </xacro:inertial_cylinder>
     </link>
-    <gazebo reference="caster_wheel">
-        <material>Gazebo/Black</material>
+    <gazebo reference="left_front_wheel">
+        <material>Gazebo/Blue</material>
+    </gazebo>
+    <!-- RIGHT FRONT WHEEL LINK -->
+    <joint name="right_front_wheel_joint" type="continuous">
+        <parent link="base_link"/>
+        <child link="right_front_wheel"/>
+        <origin xyz="0.2 -0.175 0" rpy="${pi/2} 0 0" />
+        <axis xyz="0 0 -1"/>
+    </joint>
+    <link name="right_front_wheel">
+        <visual>
+            <geometry>
+                <cylinder radius="0.04" length="0.04"/>
+            </geometry>
+            <material name="blue"/>
+        </visual>
+        <collision>
+            <geometry>
+                <cylinder radius="0.04" length="0.04"/>
+            </geometry>
+        </collision>
+        <xacro:inertial_cylinder mass="0.1" length="0.04" radius="0.05">
+            <origin xyz="0 0 0" rpy="0 0 0"/>
+        </xacro:inertial_cylinder>
+    </link>
+    <gazebo reference="right_front_wheel">
+        <material>Gazebo/Blue</material>
     </gazebo>
 </robot>

Commit message: added caster wheel

File: src/sec_bot/description/robot_core.xacro (robot description, xacro)
@@ -148,3 +148,29 @@
         <material>Gazebo/Blue</material>
     </gazebo>
+    <!-- CASTER WHEEL LINK -->
+    <joint name="caster_wheel_joint" type="continuous">
+        <parent link="base_link"/>
+        <child link="caster_wheel"/>
+        <origin xyz="0 0 0" rpy="${pi/2} 0 0" />
+        <axis xyz="0 0 0"/>
+    </joint>
+    <link name="caster_wheel">
+        <visual>
+            <geometry>
+                <cylinder radius="0.04" length="0.04"/>
+            </geometry>
+            <material name="black"/>
+        </visual>
+        <collision>
+            <geometry>
+                <cylinder radius="0.04" length="0.04"/>
+            </geometry>
+        </collision>
+        <xacro:inertial_cylinder mass="0.1" length="0.04" radius="0.05">
+            <origin xyz="0 0 0" rpy="0 0 0"/>
+        </xacro:inertial_cylinder>
+    </link>
+    <gazebo reference="right_front_wheel">
+        <material>Gazebo/Black</material>
+    </gazebo>
 </robot>

Commit message: maybe fixed cooridnates

File: src/sec_bot/description/robot_core.xacro (robot description, xacro)
@@ -152,5 +152,5 @@
         <parent link="base_link"/>
         <child link="caster_wheel"/>
-        <origin xyz="0 0 0" rpy="${pi/2} 0 0" />
+        <origin xyz="-0.01 0 0" rpy="${pi/2} 0 0" />
         <axis xyz="0 0 0"/>
     </joint>

Commit message: try again me

File: src/sec_bot/description/robot_core.xacro (robot description, xacro)
@@ -152,5 +152,5 @@
         <parent link="base_link"/>
         <child link="caster_wheel"/>
-        <origin xyz="-0.01 0 0" rpy="${pi/2} 0 0" />
+        <origin xyz="-0.1 0 0" rpy="${pi/2} 0 0" />
         <axis xyz="0 0 0"/>
     </joint>

Commit message: try again me

File: src/sec_bot/description/robot_core.xacro (robot description, xacro)
@@ -152,5 +152,5 @@
         <parent link="base_link"/>
         <child link="caster_wheel"/>
-        <origin xyz="-0.1 0 0" rpy="${pi/2} 0 0" />
+        <origin xyz="0.09 0 0" rpy="${pi/2} 0 0" />
         <axis xyz="0 0 0"/>
     </joint>

Commit message: trying to rotate the middle wheel

File: src/sec_bot/description/robot_core.xacro (robot description, xacro)
@@ -153,5 +153,5 @@
         <child link="caster_wheel"/>
         <origin xyz="0.09 0 0" rpy="${pi/2} 0 0" />
-        <axis xyz="0 0 0"/>
+        <axis xyz="0 10 0"/>
     </joint>
     <link name="caster_wheel">

Commit message: trying to rotate the middle wheel

File: src/sec_bot/description/robot_core.xacro (robot description, xacro)
@@ -152,6 +152,6 @@
         <parent link="base_link"/>
         <child link="caster_wheel"/>
-        <origin xyz="0.09 0 0" rpy="${pi/2} 0 0" />
-        <axis xyz="0 10 0"/>
+    <origin xyz="0.09 0 0" rpy="${pi/2} ${pi} 0" />
+        <axis xyz="0 0 0"/>
     </joint>
     <link name="caster_wheel">

Commit message: trying a solution from youtube

File: src/sec_bot/description/robot_core.xacro (robot description, xacro)
@@ -152,6 +152,6 @@
         <parent link="base_link"/>
         <child link="caster_wheel"/>
-    <origin xyz="0.09 0 0" rpy="${pi/2} ${pi} 0" />
-        <axis xyz="0 0 0"/>
+    <origin xyz="0.09 0 0" rpy="-${pi/2} 0 0" />
+        <axis xyz="0 0 1"/>
     </joint>
     <link name="caster_wheel">

Commit message: trying a solution from youtube

File: src/sec_bot/description/robot_core.xacro (robot description, xacro)
@@ -172,5 +172,7 @@
     </link>
     <gazebo reference="caster_wheel">
-        <material>Gazebo/Black</material>
+    <material>Gazebo/Black</material>
+    <mu1 value="0.001"/>
+    <mu2 value="0.001"/>
     </gazebo>
 </robot>

Commit message: disabling middle wheel

File: src/sec_bot/description/robot_core.xacro (robot description, xacro)
@@ -149,30 +149,32 @@
     </gazebo>
     <!-- CASTER WHEEL LINK -->
-    <joint name="caster_wheel_joint" type="continuous">
-        <parent link="base_link"/>
-        <child link="caster_wheel"/>
-    <origin xyz="0.09 0 0" rpy="-${pi/2} 0 0" />
-        <axis xyz="0 0 1"/>
-    </joint>
-    <link name="caster_wheel">
-        <visual>
-            <geometry>
-                <cylinder radius="0.04" length="0.04"/>
-            </geometry>
-            <material name="black"/>
-        </visual>
-        <collision>
-            <geometry>
-                <cylinder radius="0.04" length="0.04"/>
-            </geometry>
-        </collision>
-        <xacro:inertial_cylinder mass="0.1" length="0.04" radius="0.05">
-            <origin xyz="0 0 0" rpy="0 0 0"/>
-        </xacro:inertial_cylinder>
-    </link>
-    <gazebo reference="caster_wheel">
-    <material>Gazebo/Black</material>
-    <mu1 value="0.001"/>
-    <mu2 value="0.001"/>
-    </gazebo>
+    <!--<joint name="caster_wheel_joint" type="continuous">-->
+    <!--    <parent link="base_link"/>-->
+    <!--    <child link="caster_wheel"/>-->
+    <!--<origin xyz="0.09 0 0" rpy="-${pi/2} 0 0" />-->
+    <!--    <axis xyz="0 0 1"/>-->
+    <!--</joint>-->
+    <!---->
+    <!--<link name="caster_wheel">-->
+    <!--    <visual>-->
+    <!--        <geometry>-->
+    <!--            <cylinder radius="0.04" length="0.04"/>-->
+    <!--        </geometry>-->
+    <!--        <material name="black"/>-->
+    <!--    </visual>-->
+    <!--    <collision>-->
+    <!--        <geometry>-->
+    <!--            <cylinder radius="0.04" length="0.04"/>-->
+    <!--        </geometry>-->
+    <!--    </collision>-->
+    <!--    <xacro:inertial_cylinder mass="0.1" length="0.04" radius="0.05">-->
+    <!--        <origin xyz="0 0 0" rpy="0 0 0"/>-->
+    <!--    </xacro:inertial_cylinder>-->
+    <!--</link>-->
+    <!---->
+    <!--<gazebo reference="caster_wheel">-->
+    <!--<material>Gazebo/Black</material>-->
+    <!--<mu1 value="0.001"/>-->
+    <!--<mu2 value="0.001"/>-->
+    <!--</gazebo>-->
 </robot>

Commit message: added gazebo keyboard control

File: src/sec_bot/description/robot_core.xacro (robot description, xacro)
@@ -48,5 +48,5 @@
         <parent link="base_link"/>
         <child link="left_back_wheel"/>
-        <origin xyz="-0.02 0.175 0" rpy="-${pi/2} 0 0" />
+        <origin xyz="-0.02 0.1400242 0" rpy="-${pi/2} 0 0" />
         <axis xyz="0 0 1"/>
     </joint>
@@ -54,5 +54,5 @@
         <visual>
             <geometry>
-                <cylinder radius="0.04" length="0.04"/>
+                <cylinder radius="0.08255" length="0.020955"/>
             </geometry>
             <material name="blue"/>
@@ -60,8 +60,8 @@
         <collision>
             <geometry>
-                <cylinder radius="0.04" length="0.04"/>
+                <cylinder radius="0.08255" length="0.020955"/>
             </geometry>
         </collision>
-        <xacro:inertial_cylinder mass="0.1" length="0.04" radius="0.05">
+        <xacro:inertial_cylinder mass="0.1" length="0.020955" radius="0.08255">
             <origin xyz="0 0 0" rpy="0 0 0"/>
         </xacro:inertial_cylinder>
@@ -74,5 +74,5 @@
         <parent link="base_link"/>
         <child link="right_back_wheel"/>
-        <origin xyz="-0.02 -0.175 0" rpy="${pi/2} 0 0" />
+        <origin xyz="-0.02 -0.1400242 0" rpy="${pi/2} 0 0" />
         <axis xyz="0 0 -1"/>
     </joint>
@@ -80,5 +80,5 @@
         <visual>
             <geometry>
-                <cylinder radius="0.04" length="0.04"/>
+                <cylinder radius="0.08255" length="0.020955"/>
             </geometry>
             <material name="blue"/>
@@ -86,8 +86,8 @@
         <collision>
             <geometry>
-                <cylinder radius="0.04" length="0.04"/>
+                <cylinder radius="0.08255" length="0.020955"/>
             </geometry>
         </collision>
-        <xacro:inertial_cylinder mass="0.1" length="0.04" radius="0.05">
+        <xacro:inertial_cylinder mass="0.1" length="0.020955" radius="0.08255">
             <origin xyz="0 0 0" rpy="0 0 0"/>
         </xacro:inertial_cylinder>
@@ -100,5 +100,5 @@
         <parent link="base_link"/>
         <child link="left_front_wheel"/>
-        <origin xyz="0.2 0.175 0" rpy="-${pi/2} 0 0" />
+        <origin xyz="0.2 0.1400242 0" rpy="-${pi/2} 0 0" />
         <axis xyz="0 0 1"/>
     </joint>
@@ -106,5 +106,5 @@
         <visual>
             <geometry>
-                <cylinder radius="0.04" length="0.04"/>
+                <cylinder radius="0.08255" length="0.020955"/>
             </geometry>
             <material name="blue"/>
@@ -112,8 +112,8 @@
         <collision>
             <geometry>
-                <cylinder radius="0.04" length="0.04"/>
+                <cylinder radius="0.08255" length="0.020955"/>
             </geometry>
         </collision>
-        <xacro:inertial_cylinder mass="0.1" length="0.04" radius="0.05">
+        <xacro:inertial_cylinder mass="0.1" length="0.020955" radius="0.08255">
             <origin xyz="0 0 0" rpy="0 0 0"/>
         </xacro:inertial_cylinder>
@@ -126,5 +126,5 @@
         <parent link="base_link"/>
         <child link="right_front_wheel"/>
-        <origin xyz="0.2 -0.175 0" rpy="${pi/2} 0 0" />
+        <origin xyz="0.2 -0.1400242 0" rpy="${pi/2} 0 0" />
         <axis xyz="0 0 -1"/>
     </joint>
@@ -132,5 +132,5 @@
         <visual>
             <geometry>
-                <cylinder radius="0.04" length="0.04"/>
+                <cylinder radius="0.08255" length="0.020955"/>
             </geometry>
             <material name="blue"/>
@@ -138,8 +138,8 @@
         <collision>
             <geometry>
-                <cylinder radius="0.04" length="0.04"/>
+                <cylinder radius="0.08255" length="0.020955"/>
             </geometry>
         </collision>
-        <xacro:inertial_cylinder mass="0.1" length="0.04" radius="0.05">
+        <xacro:inertial_cylinder mass="0.1" length="0.020955" radius="0.08255">
             <origin xyz="0 0 0" rpy="0 0 0"/>
         </xacro:inertial_cylinder>
