Commit message: optimized the whole thing and added new macros

File: src/sec_bot/description/robot_core.xacro (robot description, xacro)
@@ -1,180 +1,76 @@
 <?xml version="1.0"?>
-<robot xmlns:xacro="http://www.ros.org/wiki/xacro" >
-    <xacro:include filename="inertial_macros.xacro"/>
-    <material name="white">
-        <color rgba="1 1 1 1" />
-    </material>
-    <material name="orange">
-        <color rgba="1 0.3 0.1 1"/>
-    </material>
-    <material name="blue">
-        <color rgba="0.2 0.2 1 1"/>
-    </material>
-    <material name="black">
-        <color rgba="0 0 0 1"/>
-    </material>
-    <!-- BASE LINK -->
-    <link name="base_link">
+<robot xmlns:xacro="http://www.ros.org/wiki/xacro" name="robot">
+  <!-- Includes -->
+  <xacro:include filename="inertial_macros.xacro"/>
+  <xacro:include filename="gazebo_control.xacro"/>
+  <!-- Parameters -->
+  <xacro:property name="M_PI" value="3.1415926535897931" />
+  <xacro:property name="left_back_wheel_pos" value="-0.02 0.175 0"/>
+  <xacro:property name="right_back_wheel_pos" value="-0.02 -0.175 0"/>
+  <xacro:property name="left_front_wheel_pos" value="0.2 0.175 0"/>
+  <xacro:property name="right_front_wheel_pos" value="0.2 -0.175 0"/>
+  <!-- Materials -->
+  <material name="white"><color rgba="1 1 1 1"/></material>
+  <material name="blue"><color rgba="0.2 0.2 1 1"/></material>
+  <!-- Base Structure -->
+  <link name="base_footprint"/>
+  <joint name="base_footprint_joint" type="fixed">
+    <parent link="base_footprint"/>
+    <child link="base_link"/>
+    <origin xyz="0 0 0.05"/>
+  </joint>
+  <link name="base_link"/>
+  <!-- Chassis -->
+  <joint name="chassis_joint" type="fixed">
+    <parent link="base_link"/>
+    <child link="chassis"/>
+    <origin xyz="-0.1 0 0"/>
+  </joint>
+  <link name="chassis">
+    <visual>
+      <geometry><box size="0.3 0.3 0.25"/></geometry>
+      <material name="white"/>
+    </visual>
+    <collision>
+      <geometry><box size="0.3 0.3 0.25"/></geometry>
+    </collision>
+    <xacro:inertial_box mass="0.5" x="0.3" y="0.3" z="0.25"/>
+  </link>
+  <!-- Wheels & Transmissions -->
+  <xacro:macro name="full_wheel" params="name parent origin rpy axis">
+    <joint name="${name}_joint" type="continuous">
+      <parent link="${parent}"/>
+      <child link="${name}"/>
+      <origin xyz="${origin}" rpy="${rpy}"/>
+      <axis xyz="${axis}"/>
+    </joint>
+    <link name="${name}">
+      <visual>
+        <geometry><cylinder radius="0.04" length="0.04"/></geometry>
+        <material name="blue"/>
+      </visual>
+      <collision>
+        <geometry><cylinder radius="0.04" length="0.04"/></geometry>
+      </collision>
+      <xacro:inertial_cylinder mass="0.1" radius="0.04" length="0.04"/>
     </link>
-    <!-- CHASSIS LINK -->
-    <joint name="chassis_joint" type="fixed">
-        <parent link="base_link"/>
-        <child link="chassis"/>
-        <origin xyz="-0.1 0 0"/>
-    </joint>
-    <link name="chassis">
-        <visual>
-            <origin xyz="0.19 0 0.125"/>
-            <geometry>
-                <box size="0.3 0.3 0.25"/>
-            </geometry>
-            <material name="white"/>
-        </visual>
-        <collision>
-            <origin xyz="0.19 0 0.125"/>
-            <geometry>
-                <box size="0.3 0.3 0.15"/>
-            </geometry>
-        </collision>
-        <xacro:inertial_box mass="0.5" x="0.3" y="0.3" z="0.15">
-            <origin xyz="0.15 0 0.075" rpy="0 0 0"/>
-        </xacro:inertial_box>
-    </link>
-    <gazebo reference="chassis">
-        <material>Gazebo/White</material>
-    </gazebo>
-    <!-- LEFT BACK WHEEL LINK -->
-    <joint name="left_back_wheel_joint" type="continuous">
-        <parent link="base_link"/>
-        <child link="left_back_wheel"/>
-        <origin xyz="-0.02 0.175 0" rpy="-${pi/2} 0 0" />
-        <axis xyz="0 0 1"/>
-    </joint>
-    <link name="left_back_wheel">
-        <visual>
-            <geometry>
-                <cylinder radius="0.04" length="0.04"/>
-            </geometry>
-            <material name="blue"/>
-        </visual>
-        <collision>
-            <geometry>
-                <cylinder radius="0.04" length="0.04"/>
-            </geometry>
-        </collision>
-        <xacro:inertial_cylinder mass="0.1" length="0.04" radius="0.05">
-            <origin xyz="0 0 0" rpy="0 0 0"/>
-        </xacro:inertial_cylinder>
-    </link>
-    <gazebo reference="left_back_wheel">
-        <material>Gazebo/Blue</material>
-    </gazebo>
-    <!-- RIGHT BACK WHEEL LINK -->
-    <joint name="right_back_wheel_joint" type="continuous">
-        <parent link="base_link"/>
-        <child link="right_back_wheel"/>
-        <origin xyz="-0.02 -0.175 0" rpy="${pi/2} 0 0" />
-        <axis xyz="0 0 -1"/>
-    </joint>
-    <link name="right_back_wheel">
-        <visual>
-            <geometry>
-                <cylinder radius="0.04" length="0.04"/>
-            </geometry>
-            <material name="blue"/>
-        </visual>
-        <collision>
-            <geometry>
-                <cylinder radius="0.04" length="0.04"/>
-            </geometry>
-        </collision>
-        <xacro:inertial_cylinder mass="0.1" length="0.04" radius="0.05">
-            <origin xyz="0 0 0" rpy="0 0 0"/>
-        </xacro:inertial_cylinder>
-    </link>
-    <gazebo reference="right_back_wheel">
-        <material>Gazebo/Blue</material>
-    </gazebo>
-    <!-- LEFT FRONT WHEEL LINK -->
-    <joint name="left_front_wheel_joint" type="continuous">
-        <parent link="base_link"/>
-        <child link="left_front_wheel"/>
-        <origin xyz="0.2 0.175 0" rpy="-${pi/2} 0 0" />
-        <axis xyz="0 0 1"/>
-    </joint>
-    <link name="left_front_wheel">
-        <visual>
-            <geometry>
-                <cylinder radius="0.04" length="0.04"/>
-            </geometry>
-            <material name="blue"/>
-        </visual>
-        <collision>
-            <geometry>
-                <cylinder radius="0.04" length="0.04"/>
-            </geometry>
-        </collision>
-        <xacro:inertial_cylinder mass="0.1" length="0.04" radius="0.05">
-            <origin xyz="0 0 0" rpy="0 0 0"/>
-        </xacro:inertial_cylinder>
-    </link>
-    <gazebo reference="left_front_wheel">
-        <material>Gazebo/Blue</material>
-    </gazebo>
-    <!-- RIGHT FRONT WHEEL LINK -->
-    <joint name="right_front_wheel_joint" type="continuous">
-        <parent link="base_link"/>
-        <child link="right_front_wheel"/>
-        <origin xyz="0.2 -0.175 0" rpy="${pi/2} 0 0" />
-        <axis xyz="0 0 -1"/>
-    </joint>
-    <link name="right_front_wheel">
-        <visual>
-            <geometry>
-                <cylinder radius="0.04" length="0.04"/>
-            </geometry>
-            <material name="blue"/>
-        </visual>
-        <collision>
-            <geometry>
-                <cylinder radius="0.04" length="0.04"/>
-            </geometry>
-        </collision>
-        <xacro:inertial_cylinder mass="0.1" length="0.04" radius="0.05">
-            <origin xyz="0 0 0" rpy="0 0 0"/>
-        </xacro:inertial_cylinder>
-    </link>
-    <gazebo reference="right_front_wheel">
-        <material>Gazebo/Blue</material>
-    </gazebo>
-    <!-- CASTER WHEEL LINK -->
-    <!--<joint name="caster_wheel_joint" type="continuous">-->
-    <!--    <parent link="base_link"/>-->
-    <!--    <child link="caster_wheel"/>-->
-    <!--<origin xyz="0.09 0 0" rpy="-${pi/2} 0 0" />-->
-    <!--    <axis xyz="0 0 1"/>-->
-    <!--</joint>-->
-    <!---->
-    <!--<link name="caster_wheel">-->
-    <!--    <visual>-->
-    <!--        <geometry>-->
-    <!--            <cylinder radius="0.04" length="0.04"/>-->
-    <!--        </geometry>-->
-    <!--        <material name="black"/>-->
-    <!--    </visual>-->
-    <!--    <collision>-->
-    <!--        <geometry>-->
-    <!--            <cylinder radius="0.04" length="0.04"/>-->
-    <!--        </geometry>-->
-    <!--    </collision>-->
-    <!--    <xacro:inertial_cylinder mass="0.1" length="0.04" radius="0.05">-->
-    <!--        <origin xyz="0 0 0" rpy="0 0 0"/>-->
-    <!--    </xacro:inertial_cylinder>-->
-    <!--</link>-->
-    <!---->
-    <!--<gazebo reference="caster_wheel">-->
-    <!--<material>Gazebo/Black</material>-->
-    <!--<mu1 value="0.001"/>-->
-    <!--<mu2 value="0.001"/>-->
-    <!--</gazebo>-->
+    <transmission name="${name}_trans">
+      <type>transmission_interface/SimpleTransmission</type>
+      <joint name="${name}_joint">
+        <hardwareInterface>VelocityJointInterface</hardwareInterface>
+      </joint>
+      <actuator name="${name}_motor">
+        <mechanicalReduction>1</mechanicalReduction>
+      </actuator>
+    </transmission>
+  </xacro:macro>
+  <!-- Instantiate Wheels -->
+  <xacro:full_wheel name="left_back_wheel" parent="base_link"
+                    origin="${left_back_wheel_pos}" rpy="-${M_PI/2} 0 0" axis="0 0 1"/>
+  <xacro:full_wheel name="right_back_wheel" parent="base_link"
+                    origin="${right_back_wheel_pos}" rpy="${M_PI/2} 0 0" axis="0 0 -1"/>
+  <xacro:full_wheel name="left_front_wheel" parent="base_link"
+                    origin="${left_front_wheel_pos}" rpy="-${M_PI/2} 0 0" axis="0 0 1"/>
+  <xacro:full_wheel name="right_front_wheel" parent="base_link"
+                    origin="${right_front_wheel_pos}" rpy="${M_PI/2} 0 0" axis="0 0 -1"/>
 </robot>

Commit message: passing origin xyz and rpy as single strings. please god work

File: src/sec_bot/description/robot_core.xacro (robot description, xacro)
@@ -27,14 +27,21 @@
     <origin xyz="-0.1 0 0"/>
   </joint>
-  <link name="chassis">
-    <visual>
-      <geometry><box size="0.3 0.3 0.25"/></geometry>
-      <material name="white"/>
-    </visual>
-    <collision>
-      <geometry><box size="0.3 0.3 0.25"/></geometry>
-    </collision>
-    <xacro:inertial_box mass="0.5" x="0.3" y="0.3" z="0.25"/>
-  </link>
+<link name="chassis">
+  <visual>
+    <geometry><box size="0.3 0.3 0.25"/></geometry>
+    <material name="white"/>
+  </visual>
+  <collision>
+    <geometry><box size="0.3 0.3 0.25"/></geometry>
+  </collision>
+  <xacro:inertial_box
+    mass="0.5"
+    x="0.3"
+    y="0.3"
+    z="0.25"
+    origin_xyz="'0 0 0'"
+    origin_rpy="'0 0 0'"
+  />
+</link>
   <!-- Wheels & Transmissions -->
   <xacro:macro name="full_wheel" params="name parent origin rpy axis">

Commit message: got rid of base footprint

File: src/sec_bot/description/robot_core.xacro (robot description, xacro)
@@ -14,10 +14,10 @@
   <material name="blue"><color rgba="0.2 0.2 1 1"/></material>
   <!-- Base Structure -->
-  <link name="base_footprint"/>
+  <!--- <link name="base_footprint"/>
   <joint name="base_footprint_joint" type="fixed">
     <parent link="base_footprint"/>
     <child link="base_link"/>
     <origin xyz="0 0 0.05"/>
-  </joint>
+  </joint> -->
   <link name="base_link"/>
   <!-- Chassis -->

Commit message: testing this ting

File: src/sec_bot/description/robot_core.xacro (robot description, xacro)
@@ -25,5 +25,5 @@
     <parent link="base_link"/>
     <child link="chassis"/>
-    <origin xyz="5 0 0"/>
+    <origin xyz="-0.1 0 0"/>
   </joint>
 <link name="chassis">
@@ -37,5 +37,5 @@
   <xacro:inertial_box
     mass="0.5"
-    x="0.3"
+    x="6"
     y="0.3"
     z="0.15"

Commit message: PLEASE DEEPSEEK

File: src/sec_bot/description/robot_core.xacro (robot description, xacro)
@@ -20,5 +20,18 @@
     <origin xyz="0 0 0.05"/>
   </joint> -->
-  <link name="base_link"/>
+  <link name="base_link">
+    <visual>
+      <geometry><box size="0.01 0.01 0.01"/></geometry> <!-- Small placeholder -->
+    </visual>
+    <collision>
+      <geometry><box size="0.01 0.01 0.01"/></geometry>
+    </collision>
+    <xacro:inertial_box
+      mass="0.01"  <!-- Minimal mass to avoid instability -->
+      x="0.01" y="0.01" z="0.01"
+      origin_xyz="0 0 0"
+      origin_rpy="0 0 0"
+    />
+  </link>
   <!-- Chassis -->
   <joint name="chassis_joint" type="fixed">
@@ -37,10 +50,10 @@
   <xacro:inertial_box
     mass="0.5"
-    x="6"
+    x="0.3"
     y="0.3"
     z="0.15"
     origin_xyz='0.15 0 0.075'
     origin_rpy='0 0 0'
-  />
+    />
 </link>
   <!-- Wheels & Transmissions -->

Commit message: reverted

File: src/sec_bot/description/robot_core.xacro (robot description, xacro)
@@ -20,18 +20,5 @@
     <origin xyz="0 0 0.05"/>
   </joint> -->
-  <link name="base_link">
-    <visual>
-      <geometry><box size="0.01 0.01 0.01"/></geometry> <!-- Small placeholder -->
-    </visual>
-    <collision>
-      <geometry><box size="0.01 0.01 0.01"/></geometry>
-    </collision>
-    <xacro:inertial_box
-      mass="0.01"
-      x="0.01" y="0.01" z="0.01"
-      origin_xyz="0 0 0"
-      origin_rpy="0 0 0"
-    />
-  </link>
+  <link name="base_link"/>
   <!-- Chassis -->
   <joint name="chassis_joint" type="fixed">

Commit message: lets try the french approach

File: src/sec_bot/description/robot_core.xacro (robot description, xacro)
@@ -45,10 +45,10 @@
 </link>
   <!-- Wheels & Transmissions -->
-  <xacro:macro name="full_wheel" params="name parent origin rpy axis">
+  <xacro:macro name="full_wheel" params="name parent origin rpy">
     <joint name="${name}_joint" type="continuous">
       <parent link="${parent}"/>
       <child link="${name}"/>
       <origin xyz="${origin}" rpy="${rpy}"/>
-      <axis xyz="${axis}"/>
+      <axis xyz="0 0 1"/>  <!-- Use a proper unit vector for rotation axis -->
     </joint>
     <link name="${name}">

Commit message: lets try the second french empire method

File: src/sec_bot/description/robot_core.xacro (robot description, xacro)
@@ -20,35 +20,40 @@
     <origin xyz="0 0 0.05"/>
   </joint> -->
-  <link name="base_link"/>
-  <!-- Chassis -->
+  <link name="base_link">
+    <!-- Add an empty but valid inertial element -->
+    <inertial>
+      <mass value="0.001"/>
+      <inertia ixx="0.0001" ixy="0" ixz="0" iyy="0.0001" iyz="0" izz="0.0001"/>
+    </inertial>
+  </link>
   <joint name="chassis_joint" type="fixed">
     <parent link="base_link"/>
     <child link="chassis"/>
-    <origin xyz="-0.1 0 0"/>
+    <origin xyz="-0.1 0 0.05"/>  <!-- Raise it slightly above ground -->
   </joint>
-<link name="chassis">
-  <visual>
-    <geometry><box size="0.3 0.3 0.25"/></geometry>
-    <material name="white"/>
-  </visual>
-  <collision>
-    <geometry><box size="0.3 0.3 0.25"/></geometry>
-  </collision>
-  <xacro:inertial_box
-    mass="0.5"
-    x="0.3"
-    y="0.3"
-    z="0.15"
-    origin_xyz='0.15 0 0.075'
-    origin_rpy='0 0 0'
-    />
-</link>
+  <link name="chassis">
+    <visual>
+      <geometry><box size="0.3 0.3 0.25"/></geometry>
+      <material name="white"/>
+    </visual>
+    <collision>
+      <geometry><box size="0.3 0.3 0.25"/></geometry>
+    </collision>
+    <xacro:inertial_box
+      mass="0.5"
+      x="0.3"
+      y="0.3"
+      z="0.15"
+      origin_xyz='0.15 0 0.075'
+      origin_rpy='0 0 0'
+      />
+  </link>
   <!-- Wheels & Transmissions -->
   <xacro:macro name="full_wheel" params="name parent origin rpy">
     <joint name="${name}_joint" type="continuous">
-      <parent link="${parent}"/>
-      <child link="${name}"/>
-      <origin xyz="${origin}" rpy="${rpy}"/>
-      <axis xyz="0 0 1"/>  <!-- Use a proper unit vector for rotation axis -->
+        <parent link="${parent}"/>
+        <child link="${name}"/>
+        <origin xyz="${origin}" rpy="${rpy}"/>
+        <axis xyz="0 1 0"/>  <!-- This is for wheels that rotate around Y axis -->
     </joint>
     <link name="${name}">

Commit message: twehhsfbedgsdfbgbfdsgbgfe

File: src/sec_bot/description/robot_core.xacro (robot description, xacro)
@@ -86,3 +86,34 @@
   <xacro:full_wheel name="right_front_wheel" parent="chassis"
     origin="${right_front_wheel_pos}" rpy="${M_PI/2} 0 0"/>
+  <!-- Add this to your robot_core.xacro file -->
+  <gazebo reference="chassis">
+    <material>Gazebo/White</material>
+    <mu1>0.2</mu1>
+    <mu2>0.2</mu2>
+    <selfCollide>true</selfCollide>
+  </gazebo>
+  <gazebo reference="left_back_wheel">
+    <material>Gazebo/Blue</material>
+    <mu1>1.0</mu1>
+    <mu2>1.0</mu2>
+    <selfCollide>true</selfCollide>
+  </gazebo>
+  <gazebo reference="right_back_wheel">
+    <material>Gazebo/Blue</material>
+    <mu1>1.0</mu1>
+    <mu2>1.0</mu2>
+    <selfCollide>true</selfCollide>
+  </gazebo>
+  <gazebo reference="left_front_wheel">
+    <material>Gazebo/Blue</material>
+    <mu1>1.0</mu1>
+    <mu2>1.0</mu2>
+    <selfCollide>true</selfCollide>
+  </gazebo>
+  <gazebo reference="right_front_wheel">
+    <material>Gazebo/Blue</material>
+    <mu1>1.0</mu1>
+    <mu2>1.0</mu2>
+    <selfCollide>true</selfCollide>
+  </gazebo>
 </robot>

Commit message: wethrffbsdsdbfsdbfsdfbv

File: src/sec_bot/description/robot_core.xacro (robot description, xacro)
@@ -34,18 +34,17 @@
   <link name="chassis">
     <visual>
+      <origin xyz="0 0 0.125"/>  <!-- Center the visual on the Z-axis -->
       <geometry><box size="0.3 0.3 0.25"/></geometry>
       <material name="white"/>
     </visual>
     <collision>
+      <origin xyz="0 0 0.125"/>  <!-- Center the collision on the Z-axis -->
       <geometry><box size="0.3 0.3 0.25"/></geometry>
     </collision>
-    <xacro:inertial_box
-      mass="0.5"
-      x="0.3"
-      y="0.3"
-      z="0.15"
-      origin_xyz='0.15 0 0.075'
-      origin_rpy='0 0 0'
-      />
+    <inertial>
+      <mass value="1.0"/>
+      <origin xyz="0 0 0.125"/>  <!-- Center the inertial on the Z-axis -->
+      <inertia ixx="0.015" ixy="0" ixz="0" iyy="0.0375" iyz="0" izz="0.0375"/>
+    </inertial>
   </link>
   <!-- Wheels & Transmissions -->

Commit message: trying french meeeethod

File: src/sec_bot/description/robot_core.xacro (robot description, xacro)
@@ -6,20 +6,14 @@
   <!-- Parameters -->
   <xacro:property name="M_PI" value="3.1415926535897931" />
-  <xacro:property name="left_back_wheel_pos" value="-0.02 0.175 0"/>
-  <xacro:property name="right_back_wheel_pos" value="-0.02 -0.175 0"/>
-  <xacro:property name="left_front_wheel_pos" value="0.2 0.175 0"/>
-  <xacro:property name="right_front_wheel_pos" value="0.2 -0.175 0"/>
+  <!-- Corrected wheel positions to match image -->
+  <xacro:property name="left_back_wheel_pos" value="-0.15 0.175 0"/>
+  <xacro:property name="right_back_wheel_pos" value="-0.15 -0.175 0"/>
+  <xacro:property name="left_front_wheel_pos" value="0.15 0.175 0"/>
+  <xacro:property name="right_front_wheel_pos" value="0.15 -0.175 0"/>
   <!-- Materials -->
   <material name="white"><color rgba="1 1 1 1"/></material>
   <material name="blue"><color rgba="0.2 0.2 1 1"/></material>
   <!-- Base Structure -->
-  <!--- <link name="base_footprint"/>
-  <joint name="base_footprint_joint" type="fixed">
-    <parent link="base_footprint"/>
-    <child link="base_link"/>
-    <origin xyz="0 0 0.05"/>
-  </joint> -->
   <link name="base_link">
-    <!-- Add an empty but valid inertial element -->
     <inertial>
       <mass value="0.001"/>
@@ -30,19 +24,19 @@
     <parent link="base_link"/>
     <child link="chassis"/>
-    <origin xyz="-0.1 0 0.05"/>  <!-- Raise it slightly above ground -->
+    <origin xyz="0 0 0.05"/>  <!-- Centered position to match image -->
   </joint>
   <link name="chassis">
     <visual>
-      <origin xyz="0 0 0.125"/>  <!-- Center the visual on the Z-axis -->
+      <origin xyz="0 0 0.125"/>
       <geometry><box size="0.3 0.3 0.25"/></geometry>
       <material name="white"/>
     </visual>
     <collision>
-      <origin xyz="0 0 0.125"/>  <!-- Center the collision on the Z-axis -->
+      <origin xyz="0 0 0.125"/>
       <geometry><box size="0.3 0.3 0.25"/></geometry>
     </collision>
     <inertial>
       <mass value="1.0"/>
-      <origin xyz="0 0 0.125"/>  <!-- Center the inertial on the Z-axis -->
+      <origin xyz="0 0 0.125"/>
       <inertia ixx="0.015" ixy="0" ixz="0" iyy="0.0375" iyz="0" izz="0.0375"/>
     </inertial>
@@ -58,16 +52,17 @@
     <link name="${name}">
       <visual>
-        <geometry><cylinder radius="0.04" length="0.04"/></geometry>
+        <geometry><cylinder radius="0.08255" length="0.04"/>
+        </geometry>
         <material name="blue"/>
       </visual>
       <collision>
-        <geometry><cylinder radius="0.04" length="0.04"/></geometry>
+        <geometry><cylinder radius="0.08255" length="0.04"/></geometry>
       </collision>
-      <xacro:inertial_cylinder mass="0.1" radius="0.04" length="0.04"/>
+      <xacro:inertial_cylinder mass="0.1" radius="0.08255" length="0.04"/>
     </link>
     <transmission name="${name}_trans">
       <type>transmission_interface/SimpleTransmission</type>
       <joint name="${name}_joint">
-        <hardwareInterface>VelocityJointInterface</hardwareInterface>
+        <hardwareInterface>hardware_interface/VelocityJointInterface</hardwareInterface>
       </joint>
       <actuator name="${name}_motor">
@@ -85,5 +80,5 @@
   <xacro:full_wheel name="right_front_wheel" parent="chassis"
     origin="${right_front_wheel_pos}" rpy="${M_PI/2} 0 0"/>
-  <!-- Add this to your robot_core.xacro file -->
+  <!-- Gazebo-specific properties -->
   <gazebo reference="chassis">
     <material>Gazebo/White</material>
