Commit message: trying peytons fix

File: src/sec_bot/description/robot_core.xacro (robot description, xacro)
@@ -9,5 +9,4 @@
   <!-- Parameters -->
   <xacro:property name="M_PI" value="3.1415926535897931" />
-  <!-- Wheel positions adjusted to show all 4 wheels -->
   <xacro:property name="left_back_wheel_pos" value="-0.1 0.175 0"/>
   <xacro:property name="right_back_wheel_pos" value="-0.1 -0.175 0"/>
@@ -24,5 +23,5 @@
     <parent link="base_link"/>
     <child link="chassis"/>
-    <origin xyz="0 0 0.05"/>  <!-- Centered position to match image -->
+    <origin xyz="0 0 0.05"/>
   </joint>
   <link name="chassis">
@@ -42,16 +41,15 @@
     </inertial>
   </link>
-  <!-- Wheels & Transmissions -->
+  <!-- Wheel Macro -->
   <xacro:macro name="full_wheel" params="name parent origin rpy">
     <joint name="${name}_joint" type="continuous">
-        <parent link="${parent}"/>
-        <child link="${name}"/>
-        <origin xyz="${origin}" rpy="${rpy}"/>
-        <axis xyz="0 1 0"/>  <!-- This is for wheels that rotate around Y axis -->
+      <parent link="${parent}"/>
+      <child link="${name}"/>
+      <origin xyz="${origin}" rpy="${rpy}"/>
+      <axis xyz="0 1 0"/>
     </joint>
     <link name="${name}">
       <visual>
-        <geometry><cylinder radius="0.08255" length="0.04"/>
-        </geometry>
+        <geometry><cylinder radius="0.08255" length="0.04"/></geometry>
         <material name="blue"/>
       </visual>
@@ -72,13 +70,9 @@
   </xacro:macro>
   <!-- Instantiate Wheels -->
-  <xacro:full_wheel name="left_back_wheel" parent="chassis"
-    origin="${left_back_wheel_pos}" rpy="${-(M_PI/2)} 0 0"/>
-  <xacro:full_wheel name="right_back_wheel" parent="chassis"
-    origin="${right_back_wheel_pos}" rpy="${M_PI/2} 0 0"/>
-  <xacro:full_wheel name="left_front_wheel" parent="chassis"
-    origin="${left_front_wheel_pos}" rpy="${-(M_PI/2)} 0 0"/>
-  <xacro:full_wheel name="right_front_wheel" parent="chassis"
-    origin="${right_front_wheel_pos}" rpy="${M_PI/2} 0 0"/>
-  <!-- Gazebo-specific properties -->
+  <xacro:full_wheel name="left_back_wheel" parent="chassis" origin="${left_back_wheel_pos}" rpy="${-(M_PI/2)} 0 0"/>
+  <xacro:full_wheel name="right_back_wheel" parent="chassis" origin="${right_back_wheel_pos}" rpy="${M_PI/2} 0 0"/>
+  <xacro:full_wheel name="left_front_wheel" parent="chassis" origin="${left_front_wheel_pos}" rpy="${-(M_PI/2)} 0 0"/>
+  <xacro:full_wheel name="right_front_wheel" parent="chassis" origin="${right_front_wheel_pos}" rpy="${M_PI/2} 0 0"/>
+  <!-- Gazebo Visuals -->
   <gazebo reference="chassis">
     <material>Gazebo/White</material>
@@ -111,5 +105,5 @@
     <selfCollide>true</selfCollide>
   </gazebo>
-  <!-- Camera definitions -->
+  <!-- Cameras -->
   <!-- Left Camera -->
   <joint name="camera_joint" type="fixed">
@@ -120,13 +114,9 @@
   <link name="camera_link">
     <visual>
-      <geometry>
-        <box size="0.010 0.03 0.03"/>
-      </geometry>
+      <geometry><box size="0.010 0.03 0.03"/></geometry>
       <material name="camera_red"/>
     </visual>
     <collision>
-      <geometry>
-        <box size="0.010 0.03 0.03"/>
-      </geometry>
+      <geometry><box size="0.010 0.03 0.03"/></geometry>
     </collision>
     <inertial>
@@ -140,5 +130,5 @@
     <origin xyz="0 0 0" rpy="${-M_PI/2} 0 ${-M_PI/2}"/>
   </joint>
-  <link name="camera_link_optical"></link>
+  <link name="camera_link_optical"/>
   <!-- Right Camera -->
   <joint name="camera2_joint" type="fixed">
@@ -149,13 +139,9 @@
   <link name="camera2_link">
     <visual>
-      <geometry>
-        <box size="0.010 0.03 0.03"/>
-      </geometry>
+      <geometry><box size="0.010 0.03 0.03"/></geometry>
       <material name="camera_red"/>
     </visual>
     <collision>
-      <geometry>
-        <box size="0.010 0.03 0.03"/>
-      </geometry>
+      <geometry><box size="0.010 0.03 0.03"/></geometry>
     </collision>
     <inertial>
@@ -169,11 +155,10 @@
     <origin xyz="0 0 0" rpy="${-M_PI/2} 0 ${-M_PI/2}"/>
   </joint>
-  <link name="camera2_link_optical"></link>
-  <!-- Gazebo camera plugins -->
+  <link name="camera2_link_optical"/>
+  <!-- Gazebo Harmonic Camera Sensors -->
   <gazebo reference="camera_link">
     <material>Gazebo/Red</material>
-    <sensor name="camera" type="camera">
-      <pose> 0 0 0 0 0 0 </pose>
-      <visualize>true</visualize>
+    <sensor name="camera_sensor" type="camera">
+      <pose>0 0 0 0 0 0</pose>
       <update_rate>10</update_rate>
       <camera>
@@ -189,14 +174,12 @@
         </clip>
       </camera>
-      <plugin name="camera_controller" filename="libgazebo_ros_camera.so">
-        <frame_name>camera_link_optical</frame_name>
-      </plugin>
+      <always_on>true</always_on>
+      <visualize>true</visualize>
     </sensor>
   </gazebo>
   <gazebo reference="camera2_link">
     <material>Gazebo/Red</material>
-    <sensor name="camera2" type="camera">
-      <pose> 0 0 0 0 0 0 </pose>
-      <visualize>true</visualize>
+    <sensor name="camera2_sensor" type="camera">
+      <pose>0 0 0 0 0 0</pose>
       <update_rate>10</update_rate>
       <camera>
@@ -212,7 +195,6 @@
         </clip>
       </camera>
-      <plugin name="camera2_controller" filename="libgazebo_ros_camera.so">
-        <frame_name>camera2_link_optical</frame_name>
-      </plugin>
+      <always_on>true</always_on>
+      <visualize>true</visualize>
     </sensor>
   </gazebo>
